Commit message: Add a stl version of the model.

File: romeo_description/urdf/romeo_small.urdf (robot description, URDF)
Before this commit: robot romeo, 44 links, 43 joints
Links:
- link HeadRollLink: geometry collision mesh filename=package://romeo_description/meshes/HeadRoll.stl; visual mesh filename=package://romeo_description/meshes/HeadRoll.stl
- link LElbowYawLink: geometry collision mesh filename=package://romeo_description/meshes/LElbowYaw.stl; visual mesh filename=package://romeo_description/meshes/LElbowYaw.stl
- link LHipPitchLink: geometry collision mesh filename=package://romeo_description/meshes/LHipPitch.stl; visual mesh filename=package://romeo_description/meshes/LHipPitch.stl
- link LKneePitchLink: geometry collision mesh filename=package://romeo_description/meshes/LKneePitch.stl; visual mesh filename=package://romeo_description/meshes/LKneePitch.stl
- link LShoulderYawLink: geometry collision mesh filename=package://romeo_description/meshes/LShoulderYaw.stl; visual mesh filename=package://romeo_description/meshes/LShoulderYaw.stl
- link LWristRollLink: geometry collision mesh filename=package://romeo_description/meshes/LWristRoll.stl; visual mesh filename=package://romeo_description/meshes/LWristRoll.stl
- link LWristYawLink: geometry collision mesh filename=package://romeo_description/meshes/WristYaw.stl; visual mesh filename=package://romeo_description/meshes/WristYaw.stl
- link NeckPitchLink: geometry collision mesh filename=package://romeo_description/meshes/NeckPitch.stl; visual mesh filename=package://romeo_description/meshes/NeckPitch.stl
- link RElbowYawLink: geometry collision mesh filename=package://romeo_description/meshes/RElbowYaw.stl; visual mesh filename=package://romeo_description/meshes/RElbowYaw.stl
- link RHipPitchLink: geometry collision mesh filename=package://romeo_description/meshes/RHipPitch.stl; visual mesh filename=package://romeo_description/meshes/RHipPitch.stl
- link RKneePitchLink: geometry collision mesh filename=package://romeo_description/meshes/RKneePitch.stl; visual mesh filename=package://romeo_description/meshes/RKneePitch.stl
- link RShoulderYawLink: geometry collision mesh filename=package://romeo_description/meshes/RShoulderYaw.stl; visual mesh filename=package://romeo_description/meshes/RShoulderYaw.stl
- link RWristRollLink: geometry collision mesh filename=package://romeo_description/meshes/RWristRoll.stl; visual mesh filename=package://romeo_description/meshes/RWristRoll.stl
- link RWristYawLink: geometry collision mesh filename=package://romeo_description/meshes/WristYaw.stl; visual mesh filename=package://romeo_description/meshes/WristYaw.stl
- link body: geometry collision mesh filename=package://romeo_description/meshes/Waist.stl; visual mesh filename=package://romeo_description/meshes/Waist.stl
- link l_ankle: geometry collision mesh filename=package://romeo_description/meshes/LAnkleRoll.stl; visual mesh filename=package://romeo_description/meshes/LAnkleRoll.stl
- link l_toe: geometry collision mesh filename=package://romeo_description/meshes/LToePitch.stl; visual mesh filename=package://romeo_description/meshes/LToePitch.stl
- link l_wrist: geometry collision mesh filename=package://romeo_description/meshes/LHand.stl; visual mesh filename=package://romeo_description/meshes/LHand.stl
- link r_ankle: geometry collision mesh filename=package://romeo_description/meshes/RAnkleRoll.stl; visual mesh filename=package://romeo_description/meshes/RAnkleRoll.stl
- link r_toe: geometry collision mesh filename=package://romeo_description/meshes/RToePitch.stl; visual mesh filename=package://romeo_description/meshes/RToePitch.stl
- link r_wrist: geometry collision mesh filename=package://romeo_description/meshes/RHand.stl; visual mesh filename=package://romeo_description/meshes/RHand.stl
- link torso: geometry collision mesh filename=package://romeo_description/meshes/Torso.stl; visual mesh filename=package://romeo_description/meshes/Torso.stl
