Commit message: The l/r_wrist corresponds to the last link of the arm.
Meaning, the one just before the grippers.
Also, the root joint of choice is now 'body'
(since 'body' and 'base_link' represent the same
link, we use 'body', that is not virtual).

File: romeo_description/urdf/romeo.urdf (robot description, URDF)
Before this commit: robot romeo, 37 links, 36 joints
Links:
- removed link RWristPitch_link
- added link RWristYaw_link, mass 0.07595; visual mesh filename=package://romeo_description/meshes/WristYaw.dae
- link r_wrist: mass 0.07595 -> 0.16569; geometry visual mesh filename=package://romeo_description/meshes/RHand.dae
Joints:
- joint LHipYaw: parent base_link -> body
- joint RHipYaw: parent base_link -> body
- joint RWristPitch: child RWristPitch_link -> r_wrist; parent r_wrist -> RWristYaw_link
- joint RWristYaw: child r_wrist -> RWristYaw_link
- joint TrunkYaw: parent base_link -> body

Commit message: [romeo_description] Fix collision tags in URDF.
  * Collision tags are supposed to be at the same level as the visual
    tags.
  * For now the collision meshes are the same as the visual meshes.

File: romeo_description/urdf/romeo.urdf (robot description, URDF)
Before this commit: robot romeo, 37 links, 36 joints
Links:
- link HeadRoll_link: geometry collision mesh filename=package://romeo_description/meshes/HeadRoll.dae; visual mesh filename=package://romeo_description/meshes/HeadRoll.dae
- link LElbowYaw_link: geometry collision mesh filename=package://romeo_description/meshes/LElbowYaw.dae; visual mesh filename=package://romeo_description/meshes/LElbowYaw.dae
- link LHipPitch_link: geometry collision mesh filename=package://romeo_description/meshes/LHipPitch.dae; visual mesh filename=package://romeo_description/meshes/LHipPitch.dae
- link LKneePitch_link: geometry collision mesh filename=package://romeo_description/meshes/LKneePitch.dae; visual mesh filename=package://romeo_description/meshes/LKneePitch.dae
- link LShoulderYaw_link: geometry collision mesh filename=package://romeo_description/meshes/LShoulderYaw.dae; visual mesh filename=package://romeo_description/meshes/LShoulderYaw.dae
- link LWristRoll_link: geometry collision mesh filename=package://romeo_description/meshes/LWristRoll.dae; visual mesh filename=package://romeo_description/meshes/LWristRoll.dae
- link LWristYaw_link: geometry collision mesh filename=package://romeo_description/meshes/WristYaw.dae; visual mesh filename=package://romeo_description/meshes/WristYaw.dae
- link NeckPitch_link: geometry collision mesh filename=package://romeo_description/meshes/NeckPitch.dae; visual mesh filename=package://romeo_description/meshes/NeckPitch.dae
- link RElbowYaw_link: geometry collision mesh filename=package://romeo_description/meshes/RElbowYaw.dae; visual mesh filename=package://romeo_description/meshes/RElbowYaw.dae
- link RHipPitch_link: geometry collision mesh filename=package://romeo_description/meshes/RHipPitch.dae; visual mesh filename=package://romeo_description/meshes/RHipPitch.dae
- link RKneePitch_link: geometry collision mesh filename=package://romeo_description/meshes/RKneePitch.dae; visual mesh filename=package://romeo_description/meshes/RKneePitch.dae
- link RShoulderYaw_link: geometry collision mesh filename=package://romeo_description/meshes/RShoulderYaw.dae; visual mesh filename=package://romeo_description/meshes/RShoulderYaw.dae
- link RWristRoll_link: geometry collision mesh filename=package://romeo_description/meshes/RWristRoll.dae; visual mesh filename=package://romeo_description/meshes/RWristRoll.dae
- link RWristYaw_link: geometry collision mesh filename=package://romeo_description/meshes/WristYaw.dae; visual mesh filename=package://romeo_description/meshes/WristYaw.dae
- link l_ankle: geometry collision mesh filename=package://romeo_description/meshes/LAnkleRoll.dae; visual mesh filename=package://romeo_description/meshes/LAnkleRoll.dae
- link l_toe: geometry collision mesh filename=package://romeo_description/meshes/LToePitch.dae; visual mesh filename=package://romeo_description/meshes/LToePitch.dae
- link l_wrist: geometry collision mesh filename=package://romeo_description/meshes/LHand.dae; visual mesh filename=package://romeo_description/meshes/LHand.dae
- link r_ankle: geometry collision mesh filename=package://romeo_description/meshes/RAnkleRoll.dae; visual mesh filename=package://romeo_description/meshes/RAnkleRoll.dae
- link r_toe: geometry collision mesh filename=package://romeo_description/meshes/RToePitch.dae; visual mesh filename=package://romeo_description/meshes/RToePitch.dae
- link r_wrist: geometry collision mesh filename=package://romeo_description/meshes/RHand.dae; visual mesh filename=package://romeo_description/meshes/RHand.dae
- link torso: geometry collision mesh filename=package://romeo_description/meshes/Torso.dae; visual mesh filename=package://romeo_description/meshes/Torso.dae

Commit message: Add the cameras and the gaze body.
* The gaze body is placed between the two eyes.
* The position of the 4 cameras is relative to the gaze body.
* 2x2 joints are added, corresponding to the two eyes.
  (yaw and pitch)
* The two other cameras are fixed.

File: romeo_description/urdf/romeo.urdf (robot description, URDF)
Before this commit: robot romeo, 37 links, 36 joints
Links:
- added link CameraLeft
- added link CameraLeftEye
- added link CameraRight
- added link CameraRightEye
- added link LEyePitch_link
- added link REyePitch_link
- added link gaze
Joints:
- added joint CameraLeft_joint: type fixed, parent gaze, child CameraLeft, origin xyz=-0.0021 0.055 0.0333 rpy=0 0 0
- added joint CameraRight_joint: type fixed, parent gaze, child CameraRight, origin xyz=-0.0021 -0.055 0.0333 rpy=0 0 0
- added joint LEyePitch: type revolute, parent LEyePitch_link, child CameraLeftEye, origin xyz=0 0 0 rpy=0 0 0, axis 0 1 0, limit lower=-0.349065844444444 upper=0.349065844444444 effort=0 velocity=0
- added joint LEyeYaw: type revolute, parent gaze, child LEyePitch_link, origin xyz=0 0.0325 0 rpy=0 0 0, axis 0 0 1, limit lower=-0.523598766666667 upper=0.523598766666667 effort=0 velocity=0
- added joint REyePitch: type revolute, parent REyePitch_link, child CameraRightEye, origin xyz=0 0 0 rpy=0 0 0, axis 0 1 0, limit lower=-0.349065844444444 upper=0.349065844444444 effort=0 velocity=0
- added joint REyeYaw: type revolute, parent gaze, child REyePitch_link, origin xyz=0 -0.0325 0 rpy=0 0 0, axis 0 0 1, limit lower=-0.523598766666667 upper=0.523598766666667 effort=0 velocity=0
- added joint gaze_joint: type fixed, parent HeadRoll_link, child gaze, origin xyz=0.1111 0 0.0515 rpy=0 0 0

Commit message: Add the fingers.
* For now, the phalaxes are independent.
* The dae models of the phalaxes will follow.
* The data is based on another urdf file of Aldebaran
(more up-to-date than the website).

File: romeo_description/urdf/romeo.urdf (robot description, URDF)
Before this commit: robot romeo, 44 links, 43 joints
Links:
- added link LFinger11_link, mass 0; collision mesh filename=package://romeo_description/meshes/Phalax.dae; visual mesh filename=package://romeo_description/meshes/Phalax.dae
- added link LFinger12_link, mass 0; collision mesh filename=package://romeo_description/meshes/Phalax.dae; visual mesh filename=package://romeo_description/meshes/Phalax.dae
- added link LFinger13_link, mass 0; collision mesh filename=package://romeo_description/meshes/PhalaxEnd.dae; visual mesh filename=package://romeo_description/meshes/PhalaxEnd.dae
- added link LFinger21_link, mass 0; collision mesh filename=package://romeo_description/meshes/Phalax.dae; visual mesh filename=package://romeo_description/meshes/Phalax.dae
- added link LFinger22_link, mass 0; collision mesh filename=package://romeo_description/meshes/Phalax.dae; visual mesh filename=package://romeo_description/meshes/Phalax.dae
- added link LFinger23_link, mass 0; collision mesh filename=package://romeo_description/meshes/PhalaxEnd.dae; visual mesh filename=package://romeo_description/meshes/PhalaxEnd.dae
- added link LFinger31_link, mass 0; collision mesh filename=package://romeo_description/meshes/Phalax.dae; visual mesh filename=package://romeo_description/meshes/Phalax.dae
- added link LFinger32_link, mass 0; collision mesh filename=package://romeo_description/meshes/Phalax.dae; visual mesh filename=package://romeo_description/meshes/Phalax.dae
- added link LFinger33_link, mass 0; collision mesh filename=package://romeo_description/meshes/PhalaxEnd.dae; visual mesh filename=package://romeo_description/meshes/PhalaxEnd.dae
- added link LThumb1_link, mass 0; collision mesh filename=package://romeo_description/meshes/LThumb.dae; visual mesh filename=package://romeo_description/meshes/LThumb.dae
- added link LThumb2_link, mass 0; collision mesh filename=package://romeo_description/meshes/Phalax.dae; visual mesh filename=package://romeo_description/meshes/Phalax.dae
- added link LThumb3_link, mass 0; collision mesh filename=package://romeo_description/meshes/PhalaxEnd.dae; visual mesh filename=package://romeo_description/meshes/PhalaxEnd.dae
- added link RFinger11_link, mass 0; collision mesh filename=package://romeo_description/meshes/Phalax.dae; visual mesh filename=package://romeo_description/meshes/Phalax.dae
- added link RFinger12_link, mass 0; collision mesh filename=package://romeo_description/meshes/Phalax.dae; visual mesh filename=package://romeo_description/meshes/Phalax.dae
- added link RFinger13_link, mass 0; collision mesh filename=package://romeo_description/meshes/PhalaxEnd.dae; visual mesh filename=package://romeo_description/meshes/PhalaxEnd.dae
- added link RFinger21_link, mass 0; collision mesh filename=package://romeo_description/meshes/Phalax.dae; visual mesh filename=package://romeo_description/meshes/Phalax.dae
- added link RFinger22_link, mass 0; collision mesh filename=package://romeo_description/meshes/Phalax.dae; visual mesh filename=package://romeo_description/meshes/Phalax.dae
- added link RFinger23_link, mass 0; collision mesh filename=package://romeo_description/meshes/PhalaxEnd.dae; visual mesh filename=package://romeo_description/meshes/PhalaxEnd.dae
- added link RFinger31_link, mass 0; collision mesh filename=package://romeo_description/meshes/Phalax.dae; visual mesh filename=package://romeo_description/meshes/Phalax.dae
- added link RFinger32_link, mass 0; collision mesh filename=package://romeo_description/meshes/Phalax.dae; visual mesh filename=package://romeo_description/meshes/Phalax.dae
- added link RFinger33_link, mass 0; collision mesh filename=package://romeo_description/meshes/PhalaxEnd.dae; visual mesh filename=package://romeo_description/meshes/PhalaxEnd.dae
- added link RThumb1_link, mass 0; collision mesh filename=package://romeo_description/meshes/RThumb.dae; visual mesh filename=package://romeo_description/meshes/RThumb.dae
- added link RThumb2_link, mass 0; collision mesh filename=package://romeo_description/meshes/Phalax.dae; visual mesh filename=package://romeo_description/meshes/Phalax.dae
- added link RThumb3_link, mass 0; collision mesh filename=package://romeo_description/meshes/PhalaxEnd.dae; visual mesh filename=package://romeo_description/meshes/PhalaxEnd.dae
- link l_wrist: geometry collision mesh filename=package://romeo_description/meshes/LWristPitch.dae; visual mesh filename=package://romeo_description/meshes/LWristPitch.dae
- link r_wrist: geometry collision mesh filename=package://romeo_description/meshes/RWristPitch.dae; visual mesh filename=package://romeo_description/meshes/RWristPitch.dae
Joints:
- added joint LFinger11: type revolute, parent l_wrist, child LFinger11_link, origin xyz=0.10937 0.02468 0.00329 rpy=2.98023e-08 1.06465 0.122173, axis 0.121869 -0.992546 -4.37114e-08, limit lower=0 upper=1.06465082555556 effort=30 velocity=0
- added joint LFinger12: type revolute, parent LFinger11_link, child LFinger12_link, origin xyz=0.01818 0 0 rpy=4.64506e-08 1.06465 7.88574e-08, axis 0 -1 -4.37114e-08, limit lower=0 upper=1.06465082555556 effort=30 velocity=0
- added joint LFinger13: type revolute, parent LFinger12_link, child LFinger13_link, origin xyz=0.01818 0 0 rpy=4.64506e-08 1.06465 7.88574e-08, axis 0 -1 -4.37114e-08, limit lower=0 upper=1.06465082555556 effort=30 velocity=0
- added joint LFinger21: type revolute, parent l_wrist, child LFinger21_link, origin xyz=0.11525 0 0.00329 rpy=4.64506e-08 1.06465 7.88574e-08, axis 0 -1 -4.37114e-08, limit lower=0 upper=1.06465082555556 effort=30 velocity=0
- added joint LFinger22: type revolute, parent LFinger21_link, child LFinger22_link, origin xyz=0.01818 0 0 rpy=4.64506e-08 1.06465 7.88574e-08, axis 0 -1 -4.37114e-08, limit lower=0 upper=1.06465082555556 effort=30 velocity=0
- added joint LFinger23: type revolute, parent LFinger22_link, child LFinger23_link, origin xyz=0.01818 0 0 rpy=4.64506e-08 1.06465 7.88574e-08, axis 0 -1 -4.37114e-08, limit lower=0 upper=1.06465082555556 effort=30 velocity=0
- added joint LFinger31: type revolute, parent l_wrist, child LFinger31_link, origin xyz=0.09936 -0.02478 0.00329 rpy=3.72529e-08 1.06465 -0.122173, axis -0.121869 -0.992546 -4.37114e-08, limit lower=0 upper=1.06465082555556 effort=30 velocity=0
- added joint LFinger32: type revolute, parent LFinger31_link, child LFinger32_link, origin xyz=0.01818 0 0 rpy=4.64506e-08 1.06465 7.88574e-08, axis 0 -1 -4.37114e-08, limit lower=0 upper=1.06465082555556 effort=30 velocity=0
- added joint LFinger33: type revolute, parent LFinger32_link, child LFinger33_link, origin xyz=0.01818 0 0 rpy=4.64506e-08 1.06465 7.88574e-08, axis 0 -1 -4.37114e-08, limit lower=0 upper=1.06465082555556 effort=30 velocity=0
- added joint LThumb1: type revolute, parent l_wrist, child LThumb1_link, origin xyz=0.07115 -0.02465 -0.01233 rpy=-4.76837e-07 1.37881 -2.53073, axis -0.573576 0.819152 1.05097e-07, limit lower=0 upper=1.06465082555556 effort=30 velocity=0
- added joint LThumb2: type revolute, parent LThumb1_link, child LThumb2_link, origin xyz=0.01818 0 0 rpy=4.64506e-08 1.06465 7.88574e-08, axis 0 -1 -4.37114e-08, limit lower=0 upper=1.06465082555556 effort=30 velocity=0
- added joint LThumb3: type revolute, parent LThumb2_link, child LThumb3_link, origin xyz=0.01818 0 0 rpy=4.64506e-08 1.06465 7.88574e-08, axis 0 -1 -4.37114e-08, limit lower=0 upper=1.06465082555556 effort=30 velocity=0
- added joint RFinger11: type revolute, parent r_wrist, child RFinger11_link, origin xyz=0.10937 -0.02468 0.00329 rpy=3.72529e-08 1.06465 -0.122173, axis -0.121869 -0.992546 -4.37114e-08, limit lower=0 upper=1.06465082555556 effort=30 velocity=0
- added joint RFinger12: type revolute, parent RFinger11_link, child RFinger12_link, origin xyz=0.01818 0 0 rpy=4.64506e-08 1.06465 7.88574e-08, axis 0 -1 -4.37114e-08, limit lower=0 upper=1.06465082555556 effort=30 velocity=0
- added joint RFinger13: type revolute, parent RFinger12_link, child RFinger13_link, origin xyz=0.01818 0 0 rpy=4.64506e-08 1.06465 7.88574e-08, axis 0 -1 -4.37114e-08, limit lower=0 upper=1.06465082555556 effort=30 velocity=0
- added joint RFinger21: type revolute, parent r_wrist, child RFinger21_link, origin xyz=0.11525 0 0.00329 rpy=4.64506e-08 1.06465 7.88574e-08, axis 0 -1 -4.37114e-08, limit lower=0 upper=1.06465082555556 effort=30 velocity=0
- added joint RFinger22: type revolute, parent RFinger21_link, child RFinger22_link, origin xyz=0.01818 0 0 rpy=4.64506e-08 1.06465 7.88574e-08, axis 0 -1 -4.37114e-08, limit lower=0 upper=1.06465082555556 effort=30 velocity=0
- added joint RFinger23: type revolute, parent RFinger22_link, child RFinger23_link, origin xyz=0.01818 0 0 rpy=4.64506e-08 1.06465 7.88574e-08, axis 0 -1 -4.37114e-08, limit lower=0 upper=1.06465082555556 effort=30 velocity=0
- added joint RFinger31: type revolute, parent r_wrist, child RFinger31_link, origin xyz=0.09936 0.02478 0.00329 rpy=2.98023e-08 1.06465 0.122173, axis 0.121869 -0.992546 -4.37114e-08, limit lower=0 upper=1.06465082555556 effort=30 velocity=0
- added joint RFinger32: type revolute, parent RFinger31_link, child RFinger32_link, origin xyz=0.01818 0 0 rpy=4.64506e-08 1.06465 7.88574e-08, axis 0 -1 -4.37114e-08, limit lower=0 upper=1.06465082555556 effort=30 velocity=0
- added joint RFinger33: type revolute, parent RFinger32_link, child RFinger33_link, origin xyz=0.01818 0 0 rpy=4.64506e-08 1.06465 7.88574e-08, axis 0 -1 -4.37114e-08, limit lower=0 upper=1.06465082555556 effort=30 velocity=0
- added joint RThumb1: type revolute, parent r_wrist, child RThumb1_link, origin xyz=0.07115 0.02465 -0.01233 rpy=-2.68221e-07 1.37881 2.53073, axis 0.573576 0.819152 1.05097e-07, limit lower=0 upper=1.06465082555556 effort=30 velocity=0
- added joint RThumb2: type revolute, parent RThumb1_link, child RThumb2_link, origin xyz=0.01818 0 0 rpy=4.64506e-08 1.06465 7.88574e-08, axis 0 -1 -4.37114e-08, limit lower=0 upper=1.06465082555556 effort=30 velocity=0
- added joint RThumb3: type revolute, parent RThumb2_link, child RThumb3_link, origin xyz=0.01818 0 0 rpy=4.64506e-08 1.06465 7.88574e-08, axis 0 -1 -4.37114e-08, limit lower=0 upper=1.06465082555556 effort=30 velocity=0

Commit message: All the dof of the hands are synchronized.

File: romeo_description/urdf/romeo.urdf (robot description, URDF)
Before this commit: robot romeo, 68 links, 67 joints
Joints:
- joint LFinger12: mimic (none) -> joint=LFinger11 multiplier=1 offset=0
- joint LFinger13: mimic (none) -> joint=LFinger11 multiplier=1 offset=0
- joint LFinger21: mimic (none) -> joint=LFinger11 multiplier=1 offset=0
- joint LFinger22: mimic (none) -> joint=LFinger11 multiplier=1 offset=0
- joint LFinger23: mimic (none) -> joint=LFinger11 multiplier=1 offset=0
- joint LFinger31: mimic (none) -> joint=LFinger11 multiplier=1 offset=0
- joint LFinger32: mimic (none) -> joint=LFinger11 multiplier=1 offset=0
- joint LFinger33: mimic (none) -> joint=LFinger11 multiplier=1 offset=0
- joint LThumb1: mimic (none) -> joint=LFinger11 multiplier=1 offset=0
- joint LThumb2: mimic (none) -> joint=LFinger11 multiplier=1 offset=0
- joint LThumb3: mimic (none) -> joint=LFinger11 multiplier=1 offset=0
- joint RFinger12: mimic (none) -> joint=RFinger11 multiplier=1 offset=0
- joint RFinger13: mimic (none) -> joint=RFinger11 multiplier=1 offset=0
- joint RFinger21: mimic (none) -> joint=RFinger11 multiplier=1 offset=0
- joint RFinger22: mimic (none) -> joint=RFinger11 multiplier=1 offset=0
- joint RFinger23: mimic (none) -> joint=RFinger11 multiplier=1 offset=0
- joint RFinger31: mimic (none) -> joint=RFinger11 multiplier=1 offset=0
- joint RFinger32: mimic (none) -> joint=RFinger11 multiplier=1 offset=0
- joint RFinger33: mimic (none) -> joint=RFinger11 multiplier=1 offset=0
- joint RThumb1: mimic (none) -> joint=RFinger11 multiplier=1 offset=0
- joint RThumb2: mimic (none) -> joint=RFinger11 multiplier=1 offset=0
- joint RThumb3: mimic (none) -> joint=RFinger11 multiplier=1 offset=0

Commit message: Update the collada model of Romeo.
The robot parts now have more colors.
The textures on the torso and the head are not handled yet.
The torso and the waist have been separated. The urdf
has been modified accordingly.

File: romeo_description/urdf/romeo.urdf (robot description, URDF)
Before this commit: robot romeo, 68 links, 67 joints
Links:
- link body: geometry collision mesh filename=package://romeo_description/meshes/Waist.dae; visual mesh filename=package://romeo_description/meshes/Waist.dae
