Commit message: Use Aldebaran notations for links' name.

File: romeo_description/urdf/romeo.urdf (robot description, URDF)
Before this commit: robot romeo, 68 links, 67 joints
Links:
- removed link HeadPitch_link
- removed link HeadRoll_link
- removed link LAnklePitch_link
- removed link LElbowRoll_link
- removed link LElbowYaw_link
- removed link LFinger11_link
- removed link LFinger12_link
- removed link LFinger13_link
- removed link LFinger21_link
- removed link LFinger22_link
- removed link LFinger23_link
- removed link LFinger31_link
- removed link LFinger32_link
- removed link LFinger33_link
- removed link LHipPitch_link
- removed link LHipRoll_link
- removed link LHipYaw_link
- removed link LKneePitch_link
- removed link LShoulderPitch_link
- removed link LShoulderYaw_link
- removed link LThumb1_link
- removed link LThumb2_link
- removed link LThumb3_link
- removed link LWristRoll_link
- removed link LWristYaw_link
- removed link NeckPitch_link
- removed link NeckYaw_link
- removed link RAnklePitch_link
- removed link RElbowRoll_link
- removed link RElbowYaw_link
- removed link RFinger11_link
- removed link RFinger12_link
- removed link RFinger13_link
- removed link RFinger21_link
- removed link RFinger22_link
- removed link RFinger23_link
- removed link RFinger31_link
- removed link RFinger32_link
- removed link RFinger33_link
- removed link RHipPitch_link
- removed link RHipRoll_link
- removed link RHipYaw_link
- removed link RKneePitch_link
- removed link RShoulderPitch_link
- removed link RShoulderYaw_link
- removed link RThumb1_link
- removed link RThumb2_link
- removed link RThumb3_link
- removed link RWristRoll_link
- removed link RWristYaw_link
- added link HeadPitchLink, mass 0.13981
- added link HeadRollLink, mass 1.41282; collision mesh filename=package://romeo_description/meshes/HeadRoll.dae; visual mesh filename=package://romeo_description/meshes/HeadRoll.dae
- added link LAnklePitchLink, mass 0.5008
- added link LElbowRollLink, mass 0.39848
- added link LElbowYawLink, mass 0.31265; collision mesh filename=package://romeo_description/meshes/LElbowYaw.dae; visual mesh filename=package://romeo_description/meshes/LElbowYaw.dae
- added link LFinger11Link, mass 0; collision mesh filename=package://romeo_description/meshes/Phalax.dae; visual mesh filename=package://romeo_description/meshes/Phalax.dae
- added link LFinger12Link, mass 0; collision mesh filename=package://romeo_description/meshes/Phalax.dae; visual mesh filename=package://romeo_description/meshes/Phalax.dae
- added link LFinger13Link, mass 0; collision mesh filename=package://romeo_description/meshes/PhalaxEnd.dae; visual mesh filename=package://romeo_description/meshes/PhalaxEnd.dae
- added link LFinger21Link, mass 0; collision mesh filename=package://romeo_description/meshes/Phalax.dae; visual mesh filename=package://romeo_description/meshes/Phalax.dae
- added link LFinger22Link, mass 0; collision mesh filename=package://romeo_description/meshes/Phalax.dae; visual mesh filename=package://romeo_description/meshes/Phalax.dae
- added link LFinger23Link, mass 0; collision mesh filename=package://romeo_description/meshes/PhalaxEnd.dae; visual mesh filename=package://romeo_description/meshes/PhalaxEnd.dae
- added link LFinger31Link, mass 0; collision mesh filename=package://romeo_description/meshes/Phalax.dae; visual mesh filename=package://romeo_description/meshes/Phalax.dae
- added link LFinger32Link, mass 0; collision mesh filename=package://romeo_description/meshes/Phalax.dae; visual mesh filename=package://romeo_description/meshes/Phalax.dae
- added link LFinger33Link, mass 0; collision mesh filename=package://romeo_description/meshes/PhalaxEnd.dae; visual mesh filename=package://romeo_description/meshes/PhalaxEnd.dae
- added link LHipPitchLink, mass 4.33935; collision mesh filename=package://romeo_description/meshes/LHipPitch.dae; visual mesh filename=package://romeo_description/meshes/LHipPitch.dae
- added link LHipRollLink, mass 0.6607
- added link LHipYawLink, mass 0.49477
- added link LKneePitchLink, mass 2.61063; collision mesh filename=package://romeo_description/meshes/LKneePitch.dae; visual mesh filename=package://romeo_description/meshes/LKneePitch.dae
- added link LShoulderPitchLink, mass 0.69402
- added link LShoulderYawLink, mass 0.57151; collision mesh filename=package://romeo_description/meshes/LShoulderYaw.dae; visual mesh filename=package://romeo_description/meshes/LShoulderYaw.dae
- added link LThumb1Link, mass 0; collision mesh filename=package://romeo_description/meshes/LThumb.dae; visual mesh filename=package://romeo_description/meshes/LThumb.dae
- added link LThumb2Link, mass 0; collision mesh filename=package://romeo_description/meshes/Phalax.dae; visual mesh filename=package://romeo_description/meshes/Phalax.dae
- added link LThumb3Link, mass 0; collision mesh filename=package://romeo_description/meshes/PhalaxEnd.dae; visual mesh filename=package://romeo_description/meshes/PhalaxEnd.dae
- added link LWristRollLink, mass 0.17563; collision mesh filename=package://romeo_description/meshes/LWristRoll.dae; visual mesh filename=package://romeo_description/meshes/LWristRoll.dae
- added link LWristYawLink, mass 0.07595; collision mesh filename=package://romeo_description/meshes/WristYaw.dae; visual mesh filename=package://romeo_description/meshes/WristYaw.dae
- added link NeckPitchLink, mass 0.23875; collision mesh filename=package://romeo_description/meshes/NeckPitch.dae; visual mesh filename=package://romeo_description/meshes/NeckPitch.dae
- added link NeckYawLink, mass 0.51016
- added link RAnklePitchLink, mass 0.5008
- added link RElbowRollLink, mass 0.39848
- added link RElbowYawLink, mass 0.31403; collision mesh filename=package://romeo_description/meshes/RElbowYaw.dae; visual mesh filename=package://romeo_description/meshes/RElbowYaw.dae
- added link RFinger11Link, mass 0; collision mesh filename=package://romeo_description/meshes/Phalax.dae; visual mesh filename=package://romeo_description/meshes/Phalax.dae
- added link RFinger12Link, mass 0; collision mesh filename=package://romeo_description/meshes/Phalax.dae; visual mesh filename=package://romeo_description/meshes/Phalax.dae
- added link RFinger13Link, mass 0; collision mesh filename=package://romeo_description/meshes/PhalaxEnd.dae; visual mesh filename=package://romeo_description/meshes/PhalaxEnd.dae
- added link RFinger21Link, mass 0; collision mesh filename=package://romeo_description/meshes/Phalax.dae; visual mesh filename=package://romeo_description/meshes/Phalax.dae
- added link RFinger22Link, mass 0; collision mesh filename=package://romeo_description/meshes/Phalax.dae; visual mesh filename=package://romeo_description/meshes/Phalax.dae
- added link RFinger23Link, mass 0; collision mesh filename=package://romeo_description/meshes/PhalaxEnd.dae; visual mesh filename=package://romeo_description/meshes/PhalaxEnd.dae
- added link RFinger31Link, mass 0; collision mesh filename=package://romeo_description/meshes/Phalax.dae; visual mesh filename=package://romeo_description/meshes/Phalax.dae
- added link RFinger32Link, mass 0; collision mesh filename=package://romeo_description/meshes/Phalax.dae; visual mesh filename=package://romeo_description/meshes/Phalax.dae
- added link RFinger33Link, mass 0; collision mesh filename=package://romeo_description/meshes/PhalaxEnd.dae; visual mesh filename=package://romeo_description/meshes/PhalaxEnd.dae
- added link RHipPitchLink, mass 4.33935; collision mesh filename=package://romeo_description/meshes/RHipPitch.dae; visual mesh filename=package://romeo_description/meshes/RHipPitch.dae
- added link RHipRollLink, mass 0.6607
- added link RHipYawLink, mass 0.49477
- added link RKneePitchLink, mass 2.61063; collision mesh filename=package://romeo_description/meshes/RKneePitch.dae; visual mesh filename=package://romeo_description/meshes/RKneePitch.dae
- added link RShoulderPitchLink, mass 0.69402
- added link RShoulderYawLink, mass 0.57071; collision mesh filename=package://romeo_description/meshes/RShoulderYaw.dae; visual mesh filename=package://romeo_description/meshes/RShoulderYaw.dae
- added link RThumb1Link, mass 0; collision mesh filename=package://romeo_description/meshes/RThumb.dae; visual mesh filename=package://romeo_description/meshes/RThumb.dae
- added link RThumb2Link, mass 0; collision mesh filename=package://romeo_description/meshes/Phalax.dae; visual mesh filename=package://romeo_description/meshes/Phalax.dae
- added link RThumb3Link, mass 0; collision mesh filename=package://romeo_description/meshes/PhalaxEnd.dae; visual mesh filename=package://romeo_description/meshes/PhalaxEnd.dae
- added link RWristRollLink, mass 0.17563; collision mesh filename=package://romeo_description/meshes/RWristRoll.dae; visual mesh filename=package://romeo_description/meshes/RWristRoll.dae
- added link RWristYawLink, mass 0.07595; collision mesh filename=package://romeo_description/meshes/WristYaw.dae; visual mesh filename=package://romeo_description/meshes/WristYaw.dae
Joints:
- joint HeadPitch: child HeadPitch_link -> HeadPitchLink; parent NeckPitch_link -> NeckPitchLink
- joint HeadRoll: child HeadRoll_link -> HeadRollLink; parent HeadPitch_link -> HeadPitchLink
- joint LAnklePitch: child LAnklePitch_link -> LAnklePitchLink; parent LKneePitch_link -> LKneePitchLink
- joint LAnkleRoll: parent LAnklePitch_link -> LAnklePitchLink
- joint LElbowRoll: child LElbowRoll_link -> LElbowRollLink; parent LShoulderYaw_link -> LShoulderYawLink
- joint LElbowYaw: child LElbowYaw_link -> LElbowYawLink; parent LElbowRoll_link -> LElbowRollLink
- joint LFinger11: child LFinger11_link -> LFinger11Link
- joint LFinger12: child LFinger12_link -> LFinger12Link; parent LFinger11_link -> LFinger11Link
- joint LFinger13: child LFinger13_link -> LFinger13Link; parent LFinger12_link -> LFinger12Link
- joint LFinger21: child LFinger21_link -> LFinger21Link
- joint LFinger22: child LFinger22_link -> LFinger22Link; parent LFinger21_link -> LFinger21Link
- joint LFinger23: child LFinger23_link -> LFinger23Link; parent LFinger22_link -> LFinger22Link
- joint LFinger31: child LFinger31_link -> LFinger31Link
- joint LFinger32: child LFinger32_link -> LFinger32Link; parent LFinger31_link -> LFinger31Link
- joint LFinger33: child LFinger33_link -> LFinger33Link; parent LFinger32_link -> LFinger32Link
- joint LHipPitch: child LHipPitch_link -> LHipPitchLink; parent LHipRoll_link -> LHipRollLink
- joint LHipRoll: child LHipRoll_link -> LHipRollLink; parent LHipYaw_link -> LHipYawLink
- joint LHipYaw: child LHipYaw_link -> LHipYawLink
- joint LKneePitch: child LKneePitch_link -> LKneePitchLink; parent LHipPitch_link -> LHipPitchLink
- joint LShoulderPitch: child LShoulderPitch_link -> LShoulderPitchLink
- joint LShoulderYaw: child LShoulderYaw_link -> LShoulderYawLink; parent LShoulderPitch_link -> LShoulderPitchLink
- joint LThumb1: child LThumb1_link -> LThumb1Link
- joint LThumb2: child LThumb2_link -> LThumb2Link; parent LThumb1_link -> LThumb1Link
- joint LThumb3: child LThumb3_link -> LThumb3Link; parent LThumb2_link -> LThumb2Link
- joint LWristPitch: parent LWristYaw_link -> LWristYawLink
- joint LWristRoll: child LWristRoll_link -> LWristRollLink; parent LElbowYaw_link -> LElbowYawLink
- joint LWristYaw: child LWristYaw_link -> LWristYawLink; parent LWristRoll_link -> LWristRollLink
- joint NeckPitch: child NeckPitch_link -> NeckPitchLink; parent NeckYaw_link -> NeckYawLink
- joint NeckYaw: child NeckYaw_link -> NeckYawLink
- joint RAnklePitch: child RAnklePitch_link -> RAnklePitchLink; parent RKneePitch_link -> RKneePitchLink
- joint RAnkleRoll: parent RAnklePitch_link -> RAnklePitchLink
- joint RElbowRoll: child RElbowRoll_link -> RElbowRollLink; parent RShoulderYaw_link -> RShoulderYawLink
- joint RElbowYaw: child RElbowYaw_link -> RElbowYawLink; parent RElbowRoll_link -> RElbowRollLink
- joint RFinger11: child RFinger11_link -> RFinger11Link
- joint RFinger12: child RFinger12_link -> RFinger12Link; parent RFinger11_link -> RFinger11Link
- joint RFinger13: child RFinger13_link -> RFinger13Link; parent RFinger12_link -> RFinger12Link
- joint RFinger21: child RFinger21_link -> RFinger21Link
- joint RFinger22: child RFinger22_link -> RFinger22Link; parent RFinger21_link -> RFinger21Link
- joint RFinger23: child RFinger23_link -> RFinger23Link; parent RFinger22_link -> RFinger22Link
- joint RFinger31: child RFinger31_link -> RFinger31Link
- joint RFinger32: child RFinger32_link -> RFinger32Link; parent RFinger31_link -> RFinger31Link
- joint RFinger33: child RFinger33_link -> RFinger33Link; parent RFinger32_link -> RFinger32Link
- joint RHipPitch: child RHipPitch_link -> RHipPitchLink; parent RHipRoll_link -> RHipRollLink
- joint RHipRoll: child RHipRoll_link -> RHipRollLink; parent RHipYaw_link -> RHipYawLink
- joint RHipYaw: child RHipYaw_link -> RHipYawLink
- joint RKneePitch: child RKneePitch_link -> RKneePitchLink; parent RHipPitch_link -> RHipPitchLink
- joint RShoulderPitch: child RShoulderPitch_link -> RShoulderPitchLink
- joint RShoulderYaw: child RShoulderYaw_link -> RShoulderYawLink; parent RShoulderPitch_link -> RShoulderPitchLink
- joint RThumb1: child RThumb1_link -> RThumb1Link
- joint RThumb2: child RThumb2_link -> RThumb2Link; parent RThumb1_link -> RThumb1Link
- joint RThumb3: child RThumb3_link -> RThumb3Link; parent RThumb2_link -> RThumb2Link
- joint RWristPitch: parent RWristYaw_link -> RWristYawLink
- joint RWristRoll: child RWristRoll_link -> RWristRollLink; parent RElbowYaw_link -> RElbowYawLink
- joint RWristYaw: child RWristYaw_link -> RWristYawLink; parent RWristRoll_link -> RWristRollLink
- joint gaze_joint: parent HeadRoll_link -> HeadRollLink

Commit message: Correct the way the Thumb bend.

File: romeo_description/urdf/romeo.urdf (robot description, URDF)
Before this commit: robot romeo, 68 links, 67 joints
Joints:
- joint LThumb1: limit lower=0 upper=1.06465082555556 effort=30 velocity=0 -> lower=-1.06465082555556 upper=0 effort=30 velocity=0; mimic joint=LFinger11 multiplier=1 offset=0 -> joint=LFinger11 multiplier=-1 offset=0
- joint RThumb1: limit lower=0 upper=1.06465082555556 effort=30 velocity=0 -> lower=-1.06465082555556 upper=0 effort=30 velocity=0; mimic joint=RFinger11 multiplier=1 offset=0 -> joint=RFinger11 multiplier=-1 offset=0
