Commit message: Add real torque limits.

File: romeo_description/urdf/romeo.urdf (robot description, URDF)
Before this commit: robot romeo, 68 links, 67 joints
Joints:
- joint HeadPitch: limit lower=-0.289724650888889 upper=0.349065844444444 effort=30 velocity=7.2988824 -> lower=-0.289724650888889 upper=0.349065844444444 effort=14.6811456 velocity=7.2988824
- joint HeadRoll: limit lower=-0.523598766666667 upper=0.523598766666667 effort=30 velocity=4.7442645 -> lower=-0.523598766666667 upper=0.523598766666667 effort=22.586421 velocity=4.7442645
- joint LAnklePitch: limit lower=-0.78539815 upper=0.523598766666667 effort=30 velocity=6.7799634 -> lower=-0.78539815 upper=0.523598766666667 effort=42.35835006 velocity=6.7799634
- joint LAnkleRoll: limit lower=-0.349065844444444 upper=0.349065844444444 effort=30 velocity=10.28929 -> lower=-0.349065844444444 upper=0.349065844444444 effort=27.911346822 velocity=10.28929
- joint LElbowRoll: limit lower=-2.60054054111111 upper=1.39626337777778 effort=30 velocity=10.333784 -> lower=-2.60054054111111 upper=1.39626337777778 effort=13.820682 velocity=10.333784
- joint LElbowYaw: limit lower=-1.5707963 upper=0.401425721111111 effort=30 velocity=10.3810644 -> lower=-1.5707963 upper=0.401425721111111 effort=13.757736 velocity=10.3810644
- joint LFinger11: limit lower=0 upper=1.06465082555556 effort=30 velocity=0 -> lower=0 upper=1.06465082555556 effort=0 velocity=0
- joint LFinger12: limit lower=0 upper=1.06465082555556 effort=30 velocity=0 -> lower=0 upper=1.06465082555556 effort=0 velocity=0
- joint LFinger13: limit lower=0 upper=1.06465082555556 effort=30 velocity=0 -> lower=0 upper=1.06465082555556 effort=0 velocity=0
- joint LFinger21: limit lower=0 upper=1.06465082555556 effort=30 velocity=0 -> lower=0 upper=1.06465082555556 effort=0 velocity=0
- joint LFinger22: limit lower=0 upper=1.06465082555556 effort=30 velocity=0 -> lower=0 upper=1.06465082555556 effort=0 velocity=0
- joint LFinger23: limit lower=0 upper=1.06465082555556 effort=30 velocity=0 -> lower=0 upper=1.06465082555556 effort=0 velocity=0
- joint LFinger31: limit lower=0 upper=1.06465082555556 effort=30 velocity=0 -> lower=0 upper=1.06465082555556 effort=0 velocity=0
- joint LFinger32: limit lower=0 upper=1.06465082555556 effort=30 velocity=0 -> lower=0 upper=1.06465082555556 effort=0 velocity=0
- joint LFinger33: limit lower=0 upper=1.06465082555556 effort=30 velocity=0 -> lower=0 upper=1.06465082555556 effort=0 velocity=0
- joint LHipPitch: limit lower=-1.71042263777778 upper=0.523598766666667 effort=30 velocity=6.7799634 -> lower=-1.71042263777778 upper=0.523598766666667 effort=42.35835006 velocity=6.7799634
- joint LHipRoll: limit lower=-0.261799383333333 upper=0.523598766666667 effort=30 velocity=10.289294 -> lower=-0.261799383333333 upper=0.523598766666667 effort=27.911346822 velocity=10.289294
- joint LHipYaw: limit lower=-0.261799383333333 upper=0.261799383333333 effort=30 velocity=8.082461 -> lower=-0.261799383333333 upper=0.261799383333333 effort=17.754 velocity=8.082461
- joint LKneePitch: limit lower=-0.0523598766666667 upper=2.25147469666667 effort=30 velocity=8.27600953 -> lower=-0.0523598766666667 upper=2.25147469666667 effort=17.350636374 velocity=8.27600953
- joint LShoulderPitch: limit lower=-1.51843642333333 upper=2.09439506666667 effort=30 velocity=6.52664058 -> lower=-1.51843642333333 upper=2.09439506666667 effort=21.882612 velocity=6.52664058
- joint LShoulderYaw: limit lower=-0.200712860555556 upper=1.43989660833333 effort=30 velocity=10.333784 -> lower=-0.200712860555556 upper=1.43989660833333 effort=13.820682 velocity=10.333784
- joint LThumb1: limit lower=-1.06465082555556 upper=0 effort=30 velocity=0 -> lower=-1.06465082555556 upper=0 effort=0 velocity=0
- joint LThumb2: limit lower=0 upper=1.06465082555556 effort=30 velocity=0 -> lower=0 upper=1.06465082555556 effort=0 velocity=0
- joint LThumb3: limit lower=0 upper=1.06465082555556 effort=30 velocity=0 -> lower=0 upper=1.06465082555556 effort=0 velocity=0
- joint LToePitch: limit lower=-0.78539815 upper=0 effort=30 velocity=0 -> lower=-0.78539815 upper=0 effort=0 velocity=0
- joint LWristPitch: limit lower=-0.977384364444444 upper=0.977384364444444 effort=30 velocity=0 -> lower=-0.977384364444444 upper=0.977384364444444 effort=0 velocity=0
- joint LWristRoll: limit lower=-3.66519136666667 upper=0.523598766666667 effort=30 velocity=0 -> lower=-3.66519136666667 upper=0.523598766666667 effort=0 velocity=0
- joint LWristYaw: limit lower=-0.488692182222222 upper=0.488692182222222 effort=30 velocity=0 -> lower=-0.488692182222222 upper=0.488692182222222 effort=0 velocity=0
- joint NeckPitch: limit lower=-0.698131688888889 upper=0.698131688888889 effort=30 velocity=6.17848 -> lower=-0.698131688888889 upper=0.698131688888889 effort=23.115708 velocity=6.17848
- joint NeckYaw: limit lower=-1.5707963 upper=1.5707963 effort=30 velocity=5.8886917 -> lower=-1.5707963 upper=1.5707963 effort=24.2532552 velocity=5.8886917
- joint RAnklePitch: limit lower=-0.78539815 upper=0.523598766666667 effort=30 velocity=6.7799634 -> lower=-0.78539815 upper=0.523598766666667 effort=42.35835006 velocity=6.7799634
- joint RAnkleRoll: limit lower=-0.349065844444444 upper=0.349065844444444 effort=30 velocity=10.28929 -> lower=-0.349065844444444 upper=0.349065844444444 effort=27.911346822 velocity=10.28929
- joint RElbowRoll: limit lower=-1.39626337777778 upper=2.60054054111111 effort=30 velocity=10.333784 -> lower=-1.39626337777778 upper=2.60054054111111 effort=13.820682 velocity=10.333784
- joint RElbowYaw: limit lower=-0.401425721111111 upper=1.5707963 effort=30 velocity=10.3810644 -> lower=-0.401425721111111 upper=1.5707963 effort=13.757736 velocity=10.3810644
- joint RFinger11: limit lower=0 upper=1.06465082555556 effort=30 velocity=0 -> lower=0 upper=1.06465082555556 effort=0 velocity=0
- joint RFinger12: limit lower=0 upper=1.06465082555556 effort=30 velocity=0 -> lower=0 upper=1.06465082555556 effort=0 velocity=0
- joint RFinger13: limit lower=0 upper=1.06465082555556 effort=30 velocity=0 -> lower=0 upper=1.06465082555556 effort=0 velocity=0
- joint RFinger21: limit lower=0 upper=1.06465082555556 effort=30 velocity=0 -> lower=0 upper=1.06465082555556 effort=0 velocity=0
- joint RFinger22: limit lower=0 upper=1.06465082555556 effort=30 velocity=0 -> lower=0 upper=1.06465082555556 effort=0 velocity=0
- joint RFinger23: limit lower=0 upper=1.06465082555556 effort=30 velocity=0 -> lower=0 upper=1.06465082555556 effort=0 velocity=0
- joint RFinger31: limit lower=0 upper=1.06465082555556 effort=30 velocity=0 -> lower=0 upper=1.06465082555556 effort=0 velocity=0
- joint RFinger32: limit lower=0 upper=1.06465082555556 effort=30 velocity=0 -> lower=0 upper=1.06465082555556 effort=0 velocity=0
- joint RFinger33: limit lower=0 upper=1.06465082555556 effort=30 velocity=0 -> lower=0 upper=1.06465082555556 effort=0 velocity=0
- joint RHipPitch: limit lower=-1.71042263777778 upper=0.523598766666667 effort=30 velocity=6.7799634 -> lower=-1.71042263777778 upper=0.523598766666667 effort=42.35835006 velocity=6.7799634
- joint RHipRoll: limit lower=-0.523598766666667 upper=0.261799383333333 effort=30 velocity=10.289294 -> lower=-0.523598766666667 upper=0.261799383333333 effort=27.911346822 velocity=10.289294
- joint RHipYaw: limit lower=-0.261799383333333 upper=0.261799383333333 effort=30 velocity=8.082461 -> lower=-0.261799383333333 upper=0.261799383333333 effort=17.754 velocity=8.082461
- joint RKneePitch: limit lower=-0.0523598766666667 upper=2.25147469666667 effort=30 velocity=8.27600953 -> lower=-0.0523598766666667 upper=2.25147469666667 effort=17.350636374 velocity=8.27600953
- joint RShoulderPitch: limit lower=-1.51843642333333 upper=2.09439506666667 effort=30 velocity=6.52664058 -> lower=-1.51843642333333 upper=2.09439506666667 effort=21.882612 velocity=6.52664058
- joint RShoulderYaw: limit lower=-1.43989660833333 upper=0.200712860555556 effort=30 velocity=10.333784 -> lower=-1.43989660833333 upper=0.200712860555556 effort=13.820682 velocity=10.333784
- joint RThumb1: limit lower=-1.06465082555556 upper=0 effort=30 velocity=0 -> lower=-1.06465082555556 upper=0 effort=0 velocity=0
- joint RThumb2: limit lower=0 upper=1.06465082555556 effort=30 velocity=0 -> lower=0 upper=1.06465082555556 effort=0 velocity=0
- joint RThumb3: limit lower=0 upper=1.06465082555556 effort=30 velocity=0 -> lower=0 upper=1.06465082555556 effort=0 velocity=0
- joint RToePitch: limit lower=-0.78539815 upper=0 effort=30 velocity=0 -> lower=-0.78539815 upper=0 effort=0 velocity=0
- joint RWristPitch: limit lower=-0.977384364444444 upper=0.977384364444444 effort=30 velocity=0 -> lower=-0.977384364444444 upper=0.977384364444444 effort=0 velocity=0
- joint RWristRoll: limit lower=-0.523598766666667 upper=3.66519136666667 effort=30 velocity=0 -> lower=-0.523598766666667 upper=3.66519136666667 effort=0 velocity=0
- joint RWristYaw: limit lower=-0.488692182222222 upper=0.488692182222222 effort=30 velocity=0 -> lower=-0.488692182222222 upper=0.488692182222222 effort=0 velocity=0
- joint TrunkYaw: limit lower=-0.78539815 upper=0.78539815 effort=30 velocity=0 -> lower=-0.78539815 upper=0.78539815 effort=0 velocity=0

File: romeo_description/urdf/romeo_small.urdf (robot description, URDF)
Before this commit: robot romeo, 44 links, 43 joints
Joints:
- joint HeadPitch: limit lower=-0.289724650888889 upper=0.349065844444444 effort=30 velocity=7.2988824 -> lower=-0.289724650888889 upper=0.349065844444444 effort=14.6811456 velocity=7.2988824
- joint HeadRoll: limit lower=-0.523598766666667 upper=0.523598766666667 effort=30 velocity=4.7442645 -> lower=-0.523598766666667 upper=0.523598766666667 effort=22.586421 velocity=4.7442645
- joint LAnklePitch: limit lower=-0.78539815 upper=0.523598766666667 effort=30 velocity=6.7799634 -> lower=-0.78539815 upper=0.523598766666667 effort=42.35835006 velocity=6.7799634
- joint LAnkleRoll: limit lower=-0.349065844444444 upper=0.349065844444444 effort=30 velocity=10.28929 -> lower=-0.349065844444444 upper=0.349065844444444 effort=27.911346822 velocity=10.28929
- joint LElbowRoll: limit lower=-2.60054054111111 upper=1.39626337777778 effort=30 velocity=10.333784 -> lower=-2.60054054111111 upper=1.39626337777778 effort=13.820682 velocity=10.333784
- joint LElbowYaw: limit lower=-1.5707963 upper=0.401425721111111 effort=30 velocity=10.3810644 -> lower=-1.5707963 upper=0.401425721111111 effort=13.757736 velocity=10.3810644
- joint LHipPitch: limit lower=-1.71042263777778 upper=0.523598766666667 effort=30 velocity=6.7799634 -> lower=-1.71042263777778 upper=0.523598766666667 effort=42.35835006 velocity=6.7799634
- joint LHipRoll: limit lower=-0.261799383333333 upper=0.523598766666667 effort=30 velocity=10.289294 -> lower=-0.261799383333333 upper=0.523598766666667 effort=27.911346822 velocity=10.289294
- joint LHipYaw: limit lower=-0.261799383333333 upper=0.261799383333333 effort=30 velocity=8.082461 -> lower=-0.261799383333333 upper=0.261799383333333 effort=17.754 velocity=8.082461
- joint LKneePitch: limit lower=-0.0523598766666667 upper=2.25147469666667 effort=30 velocity=8.27600953 -> lower=-0.0523598766666667 upper=2.25147469666667 effort=17.350636374 velocity=8.27600953
- joint LShoulderPitch: limit lower=-1.51843642333333 upper=2.09439506666667 effort=30 velocity=6.52664058 -> lower=-1.51843642333333 upper=2.09439506666667 effort=21.882612 velocity=6.52664058
- joint LShoulderYaw: limit lower=-0.200712860555556 upper=1.43989660833333 effort=30 velocity=10.333784 -> lower=-0.200712860555556 upper=1.43989660833333 effort=13.820682 velocity=10.333784
- joint LToePitch: limit lower=-0.78539815 upper=0 effort=30 velocity=0 -> lower=-0.78539815 upper=0 effort=0 velocity=0
- joint LWristPitch: limit lower=-0.977384364444444 upper=0.977384364444444 effort=30 velocity=0 -> lower=-0.977384364444444 upper=0.977384364444444 effort=0 velocity=0
- joint LWristRoll: limit lower=-3.66519136666667 upper=0.523598766666667 effort=30 velocity=0 -> lower=-3.66519136666667 upper=0.523598766666667 effort=0 velocity=0
- joint LWristYaw: limit lower=-0.488692182222222 upper=0.488692182222222 effort=30 velocity=0 -> lower=-0.488692182222222 upper=0.488692182222222 effort=0 velocity=0
- joint NeckPitch: limit lower=-0.698131688888889 upper=0.698131688888889 effort=30 velocity=6.17848 -> lower=-0.698131688888889 upper=0.698131688888889 effort=23.115708 velocity=6.17848
- joint NeckYaw: limit lower=-1.5707963 upper=1.5707963 effort=30 velocity=5.8886917 -> lower=-1.5707963 upper=1.5707963 effort=24.2532552 velocity=5.8886917
- joint RAnklePitch: limit lower=-0.78539815 upper=0.523598766666667 effort=30 velocity=6.7799634 -> lower=-0.78539815 upper=0.523598766666667 effort=42.35835006 velocity=6.7799634
- joint RAnkleRoll: limit lower=-0.349065844444444 upper=0.349065844444444 effort=30 velocity=10.28929 -> lower=-0.349065844444444 upper=0.349065844444444 effort=27.911346822 velocity=10.28929
- joint RElbowRoll: limit lower=-1.39626337777778 upper=2.60054054111111 effort=30 velocity=10.333784 -> lower=-1.39626337777778 upper=2.60054054111111 effort=13.820682 velocity=10.333784
- joint RElbowYaw: limit lower=-0.401425721111111 upper=1.5707963 effort=30 velocity=10.3810644 -> lower=-0.401425721111111 upper=1.5707963 effort=13.757736 velocity=10.3810644
- joint RHipPitch: limit lower=-1.71042263777778 upper=0.523598766666667 effort=30 velocity=6.7799634 -> lower=-1.71042263777778 upper=0.523598766666667 effort=42.35835006 velocity=6.7799634
- joint RHipRoll: limit lower=-0.523598766666667 upper=0.261799383333333 effort=30 velocity=10.289294 -> lower=-0.523598766666667 upper=0.261799383333333 effort=27.911346822 velocity=10.289294
- joint RHipYaw: limit lower=-0.261799383333333 upper=0.261799383333333 effort=30 velocity=8.082461 -> lower=-0.261799383333333 upper=0.261799383333333 effort=17.754 velocity=8.082461
- joint RKneePitch: limit lower=-0.0523598766666667 upper=2.25147469666667 effort=30 velocity=8.27600953 -> lower=-0.0523598766666667 upper=2.25147469666667 effort=17.350636374 velocity=8.27600953
- joint RShoulderPitch: limit lower=-1.51843642333333 upper=2.09439506666667 effort=30 velocity=6.52664058 -> lower=-1.51843642333333 upper=2.09439506666667 effort=21.882612 velocity=6.52664058
- joint RShoulderYaw: limit lower=-1.43989660833333 upper=0.200712860555556 effort=30 velocity=10.333784 -> lower=-1.43989660833333 upper=0.200712860555556 effort=13.820682 velocity=10.333784
- joint RToePitch: limit lower=-0.78539815 upper=0 effort=30 velocity=0 -> lower=-0.78539815 upper=0 effort=0 velocity=0
- joint RWristPitch: limit lower=-0.977384364444444 upper=0.977384364444444 effort=30 velocity=0 -> lower=-0.977384364444444 upper=0.977384364444444 effort=0 velocity=0
- joint RWristRoll: limit lower=-0.523598766666667 upper=3.66519136666667 effort=30 velocity=0 -> lower=-0.523598766666667 upper=3.66519136666667 effort=0 velocity=0
- joint RWristYaw: limit lower=-0.488692182222222 upper=0.488692182222222 effort=30 velocity=0 -> lower=-0.488692182222222 upper=0.488692182222222 effort=0 velocity=0
- joint TrunkYaw: limit lower=-0.78539815 upper=0.78539815 effort=30 velocity=0 -> lower=-0.78539815 upper=0.78539815 effort=0 velocity=0
