Commit message: fix scales

File: romeo_description/urdf/romeo.urdf (robot description, URDF)
Before this commit: robot romeo, 68 links, 67 joints
Links:
- link HeadRollLink: geometry collision mesh filename=package://romeo_description/meshes/HeadRoll.dae scale=100 100 100; visual mesh filename=package://romeo_description/meshes/HeadRoll.dae scale=100 100 100
- link LElbowYawLink: geometry collision mesh filename=package://romeo_description/meshes/LElbowYaw.dae scale=100 100 100; visual mesh filename=package://romeo_description/meshes/LElbowYaw.dae scale=100 100 100
- link LFinger11Link: geometry collision mesh filename=package://romeo_description/meshes/Phalax.dae scale=100 100 100; visual mesh filename=package://romeo_description/meshes/Phalax.dae scale=100 100 100
- link LFinger12Link: geometry collision mesh filename=package://romeo_description/meshes/Phalax.dae scale=100 100 100; visual mesh filename=package://romeo_description/meshes/Phalax.dae scale=100 100 100
- link LFinger13Link: geometry collision mesh filename=package://romeo_description/meshes/PhalaxEnd.dae scale=100 100 100; visual mesh filename=package://romeo_description/meshes/PhalaxEnd.dae scale=100 100 100
- link LFinger21Link: geometry collision mesh filename=package://romeo_description/meshes/Phalax.dae scale=100 100 100; visual mesh filename=package://romeo_description/meshes/Phalax.dae scale=100 100 100
- link LFinger22Link: geometry collision mesh filename=package://romeo_description/meshes/Phalax.dae scale=100 100 100; visual mesh filename=package://romeo_description/meshes/Phalax.dae scale=100 100 100
- link LFinger23Link: geometry collision mesh filename=package://romeo_description/meshes/PhalaxEnd.dae scale=100 100 100; visual mesh filename=package://romeo_description/meshes/PhalaxEnd.dae scale=100 100 100
- link LFinger31Link: geometry collision mesh filename=package://romeo_description/meshes/Phalax.dae scale=100 100 100; visual mesh filename=package://romeo_description/meshes/Phalax.dae scale=100 100 100
- link LFinger32Link: geometry collision mesh filename=package://romeo_description/meshes/Phalax.dae scale=100 100 100; visual mesh filename=package://romeo_description/meshes/Phalax.dae scale=100 100 100
- link LFinger33Link: geometry collision mesh filename=package://romeo_description/meshes/PhalaxEnd.dae scale=100 100 100; visual mesh filename=package://romeo_description/meshes/PhalaxEnd.dae scale=100 100 100
- link LHipPitchLink: geometry collision mesh filename=package://romeo_description/meshes/LHipPitch.dae scale=100 100 100; visual mesh filename=package://romeo_description/meshes/LHipPitch.dae scale=100 100 100
- link LKneePitchLink: geometry collision mesh filename=package://romeo_description/meshes/LKneePitch.dae scale=100 100 100; visual mesh filename=package://romeo_description/meshes/LKneePitch.dae scale=100 100 100
- link LShoulderYawLink: geometry collision mesh filename=package://romeo_description/meshes/LShoulderYaw.dae scale=100 100 100; visual mesh filename=package://romeo_description/meshes/LShoulderYaw.dae scale=100 100 100
- link LThumb1Link: geometry collision mesh filename=package://romeo_description/meshes/LThumb.dae scale=100 100 100; visual mesh filename=package://romeo_description/meshes/LThumb.dae scale=100 100 100
- link LThumb2Link: geometry collision mesh filename=package://romeo_description/meshes/Phalax.dae scale=100 100 100; visual mesh filename=package://romeo_description/meshes/Phalax.dae scale=100 100 100
- link LThumb3Link: geometry collision mesh filename=package://romeo_description/meshes/PhalaxEnd.dae scale=100 100 100; visual mesh filename=package://romeo_description/meshes/PhalaxEnd.dae scale=100 100 100
- link LWristRollLink: geometry collision mesh filename=package://romeo_description/meshes/LWristRoll.dae scale=100 100 100; visual mesh filename=package://romeo_description/meshes/LWristRoll.dae scale=100 100 100
- link LWristYawLink: geometry collision mesh filename=package://romeo_description/meshes/WristYaw.dae scale=100 100 100; visual mesh filename=package://romeo_description/meshes/WristYaw.dae scale=100 100 100
- link NeckPitchLink: geometry collision mesh filename=package://romeo_description/meshes/NeckPitch.dae scale=100 100 100; visual mesh filename=package://romeo_description/meshes/NeckPitch.dae scale=100 100 100
- link RElbowYawLink: geometry collision mesh filename=package://romeo_description/meshes/RElbowYaw.dae scale=100 100 100; visual mesh filename=package://romeo_description/meshes/RElbowYaw.dae scale=100 100 100
- link RFinger11Link: geometry collision mesh filename=package://romeo_description/meshes/Phalax.dae scale=100 100 100; visual mesh filename=package://romeo_description/meshes/Phalax.dae scale=100 100 100
- link RFinger12Link: geometry collision mesh filename=package://romeo_description/meshes/Phalax.dae scale=100 100 100; visual mesh filename=package://romeo_description/meshes/Phalax.dae scale=100 100 100
- link RFinger13Link: geometry collision mesh filename=package://romeo_description/meshes/PhalaxEnd.dae scale=100 100 100; visual mesh filename=package://romeo_description/meshes/PhalaxEnd.dae scale=100 100 100
- link RFinger21Link: geometry collision mesh filename=package://romeo_description/meshes/Phalax.dae scale=100 100 100; visual mesh filename=package://romeo_description/meshes/Phalax.dae scale=100 100 100
- link RFinger22Link: geometry collision mesh filename=package://romeo_description/meshes/Phalax.dae scale=100 100 100; visual mesh filename=package://romeo_description/meshes/Phalax.dae scale=100 100 100
- link RFinger23Link: geometry collision mesh filename=package://romeo_description/meshes/PhalaxEnd.dae scale=100 100 100; visual mesh filename=package://romeo_description/meshes/PhalaxEnd.dae scale=100 100 100
- link RFinger31Link: geometry collision mesh filename=package://romeo_description/meshes/Phalax.dae scale=100 100 100; visual mesh filename=package://romeo_description/meshes/Phalax.dae scale=100 100 100
- link RFinger32Link: geometry collision mesh filename=package://romeo_description/meshes/Phalax.dae scale=100 100 100; visual mesh filename=package://romeo_description/meshes/Phalax.dae scale=100 100 100
- link RFinger33Link: geometry collision mesh filename=package://romeo_description/meshes/PhalaxEnd.dae scale=100 100 100; visual mesh filename=package://romeo_description/meshes/PhalaxEnd.dae scale=100 100 100
- link RHipPitchLink: geometry collision mesh filename=package://romeo_description/meshes/RHipPitch.dae scale=100 100 100; visual mesh filename=package://romeo_description/meshes/RHipPitch.dae scale=100 100 100
- link RKneePitchLink: geometry collision mesh filename=package://romeo_description/meshes/RKneePitch.dae scale=100 100 100; visual mesh filename=package://romeo_description/meshes/RKneePitch.dae scale=100 100 100
- link RShoulderYawLink: geometry collision mesh filename=package://romeo_description/meshes/RShoulderYaw.dae scale=100 100 100; visual mesh filename=package://romeo_description/meshes/RShoulderYaw.dae scale=100 100 100
- link RThumb1Link: geometry collision mesh filename=package://romeo_description/meshes/RThumb.dae scale=100 100 100; visual mesh filename=package://romeo_description/meshes/RThumb.dae scale=100 100 100
- link RThumb2Link: geometry collision mesh filename=package://romeo_description/meshes/Phalax.dae scale=100 100 100; visual mesh filename=package://romeo_description/meshes/Phalax.dae scale=100 100 100
- link RThumb3Link: geometry collision mesh filename=package://romeo_description/meshes/PhalaxEnd.dae scale=100 100 100; visual mesh filename=package://romeo_description/meshes/PhalaxEnd.dae scale=100 100 100
- link RWristRollLink: geometry collision mesh filename=package://romeo_description/meshes/RWristRoll.dae scale=100 100 100; visual mesh filename=package://romeo_description/meshes/RWristRoll.dae scale=100 100 100
- link RWristYawLink: geometry collision mesh filename=package://romeo_description/meshes/WristYaw.dae scale=100 100 100; visual mesh filename=package://romeo_description/meshes/WristYaw.dae scale=100 100 100
- link body: geometry collision mesh filename=package://romeo_description/meshes/Waist.dae scale=100 100 100; visual mesh filename=package://romeo_description/meshes/Waist.dae scale=100 100 100
- link l_ankle: geometry collision mesh filename=package://romeo_description/meshes/LAnkleRoll.dae scale=100 100 100; visual mesh filename=package://romeo_description/meshes/LAnkleRoll.dae scale=100 100 100
- link l_toe: geometry collision mesh filename=package://romeo_description/meshes/LToePitch.dae scale=100 100 100; visual mesh filename=package://romeo_description/meshes/LToePitch.dae scale=100 100 100
- link l_wrist: geometry collision mesh filename=package://romeo_description/meshes/LWristPitch.dae scale=100 100 100; visual mesh filename=package://romeo_description/meshes/LWristPitch.dae scale=100 100 100
- link r_ankle: geometry collision mesh filename=package://romeo_description/meshes/RAnkleRoll.dae scale=100 100 100; visual mesh filename=package://romeo_description/meshes/RAnkleRoll.dae scale=100 100 100
- link r_toe: geometry collision mesh filename=package://romeo_description/meshes/RToePitch.dae scale=100 100 100; visual mesh filename=package://romeo_description/meshes/RToePitch.dae scale=100 100 100
- link r_wrist: geometry collision mesh filename=package://romeo_description/meshes/RWristPitch.dae scale=100 100 100; visual mesh filename=package://romeo_description/meshes/RWristPitch.dae scale=100 100 100
- link torso: geometry collision mesh filename=package://romeo_description/meshes/Torso.dae scale=100 100 100; visual mesh filename=package://romeo_description/meshes/Torso.dae scale=100 100 100

File: romeo_description/urdf/romeo_small.urdf (robot description, URDF)
Before this commit: robot romeo, 44 links, 43 joints
Links:
- link HeadRollLink: geometry collision mesh filename=package://romeo_description/meshes/HeadRoll.dae scale=100 100 100; visual mesh filename=package://romeo_description/meshes/HeadRoll.dae scale=100 100 100
- link LElbowYawLink: geometry collision mesh filename=package://romeo_description/meshes/LElbowYaw.dae scale=100 100 100; visual mesh filename=package://romeo_description/meshes/LElbowYaw.dae scale=100 100 100
- link LHipPitchLink: geometry collision mesh filename=package://romeo_description/meshes/LHipPitch.dae scale=100 100 100; visual mesh filename=package://romeo_description/meshes/LHipPitch.dae scale=100 100 100
- link LKneePitchLink: geometry collision mesh filename=package://romeo_description/meshes/LKneePitch.dae scale=100 100 100; visual mesh filename=package://romeo_description/meshes/LKneePitch.dae scale=100 100 100
- link LShoulderYawLink: geometry collision mesh filename=package://romeo_description/meshes/LShoulderYaw.dae scale=100 100 100; visual mesh filename=package://romeo_description/meshes/LShoulderYaw.dae scale=100 100 100
- link LWristRollLink: geometry collision mesh filename=package://romeo_description/meshes/LWristRoll.dae scale=100 100 100; visual mesh filename=package://romeo_description/meshes/LWristRoll.dae scale=100 100 100
- link LWristYawLink: geometry collision mesh filename=package://romeo_description/meshes/WristYaw.dae scale=100 100 100; visual mesh filename=package://romeo_description/meshes/WristYaw.dae scale=100 100 100
- link NeckPitchLink: geometry collision mesh filename=package://romeo_description/meshes/NeckPitch.dae scale=100 100 100; visual mesh filename=package://romeo_description/meshes/NeckPitch.dae scale=100 100 100
- link RElbowYawLink: geometry collision mesh filename=package://romeo_description/meshes/RElbowYaw.dae scale=100 100 100; visual mesh filename=package://romeo_description/meshes/RElbowYaw.dae scale=100 100 100
- link RHipPitchLink: geometry collision mesh filename=package://romeo_description/meshes/RHipPitch.dae scale=100 100 100; visual mesh filename=package://romeo_description/meshes/RHipPitch.dae scale=100 100 100
- link RKneePitchLink: geometry collision mesh filename=package://romeo_description/meshes/RKneePitch.dae scale=100 100 100; visual mesh filename=package://romeo_description/meshes/RKneePitch.dae scale=100 100 100
- link RShoulderYawLink: geometry collision mesh filename=package://romeo_description/meshes/RShoulderYaw.dae scale=100 100 100; visual mesh filename=package://romeo_description/meshes/RShoulderYaw.dae scale=100 100 100
- link RWristRollLink: geometry collision mesh filename=package://romeo_description/meshes/RWristRoll.dae scale=100 100 100; visual mesh filename=package://romeo_description/meshes/RWristRoll.dae scale=100 100 100
- link RWristYawLink: geometry collision mesh filename=package://romeo_description/meshes/WristYaw.dae scale=100 100 100; visual mesh filename=package://romeo_description/meshes/WristYaw.dae scale=100 100 100
- link body: geometry collision mesh filename=package://romeo_description/meshes/Waist.dae scale=100 100 100; visual mesh filename=package://romeo_description/meshes/Waist.dae scale=100 100 100
- link l_ankle: geometry collision mesh filename=package://romeo_description/meshes/LAnkleRoll.dae scale=100 100 100; visual mesh filename=package://romeo_description/meshes/LAnkleRoll.dae scale=100 100 100
- link l_toe: geometry collision mesh filename=package://romeo_description/meshes/LToePitch.dae scale=100 100 100; visual mesh filename=package://romeo_description/meshes/LToePitch.dae scale=100 100 100
- link l_wrist: geometry collision mesh filename=package://romeo_description/meshes/LHand.dae scale=100 100 100; visual mesh filename=package://romeo_description/meshes/LHand.dae scale=100 100 100
- link r_ankle: geometry collision mesh filename=package://romeo_description/meshes/RAnkleRoll.dae scale=100 100 100; visual mesh filename=package://romeo_description/meshes/RAnkleRoll.dae scale=100 100 100
- link r_toe: geometry collision mesh filename=package://romeo_description/meshes/RToePitch.dae scale=100 100 100; visual mesh filename=package://romeo_description/meshes/RToePitch.dae scale=100 100 100
- link r_wrist: geometry collision mesh filename=package://romeo_description/meshes/RHand.dae scale=100 100 100; visual mesh filename=package://romeo_description/meshes/RHand.dae scale=100 100 100
- link torso: geometry collision mesh filename=package://romeo_description/meshes/Torso.dae scale=100 100 100; visual mesh filename=package://romeo_description/meshes/Torso.dae scale=100 100 100

Commit message: Add gripper frames.

File: romeo_description/urdf/romeo.urdf (robot description, URDF)
Before this commit: robot romeo, 68 links, 67 joints
Links:
- added link l_gripper
- added link r_gripper
Joints:
- added joint l_gripper_joint: type fixed, parent l_wrist, child l_gripper, origin xyz=0.09 0 -0.02 rpy=-1.57079633 0 0
- added joint r_gripper_joint: type fixed, parent r_wrist, child r_gripper, origin xyz=0.09 0 -0.02 rpy=-1.57079633 0 0

File: romeo_description/urdf/romeo_small.urdf (robot description, URDF)
Before this commit: robot romeo, 44 links, 43 joints
Links:
- added link l_gripper
- added link r_gripper
Joints:
- added joint l_gripper_joint: type fixed, parent l_wrist, child l_gripper, origin xyz=0.09 0 -0.02 rpy=-1.57079633 0 0
- added joint r_gripper_joint: type fixed, parent r_wrist, child r_gripper, origin xyz=0.09 0 -0.02 rpy=-1.57079633 0 0
