Commit message: Update Romeo model.
Version 2014-05-22.
Main change: The order of the pitch and the yaw for the wrist is inverted.
Other change: Update of the joint limits and body parameters.

File: romeo_description/urdf/romeo.urdf (robot description, URDF)
Before this commit: robot romeo, 70 links, 69 joints
Links:
- removed link LEyePitch_link
- removed link REyePitch_link
- link RElbowYawLink: mass 0.31403 -> 0.31265
- link RShoulderYawLink: mass 0.57071 -> 0.57151
- link l_ankle: mass 0.64224 -> 1.07155
- link l_toe: mass 0.2889 -> 0.24032
- link r_ankle: mass 0.64224 -> 0.74347
- link r_toe: mass 0.2889 -> 0.24032
Joints:
- joint HeadPitch: limit lower=-0.289724650888889 upper=0.349065844444444 effort=14.6811456 velocity=7.2988824 -> lower=-0.349066 upper=0.279253 effort=2.57 velocity=1.9
- joint HeadRoll: limit lower=-0.523598766666667 upper=0.523598766666667 effort=22.586421 velocity=4.7442645 -> lower=-0.349066 upper=0.349066 effort=0.9 velocity=1.5
- joint LAnklePitch: limit lower=-0.78539815 upper=0.523598766666667 effort=42.35835006 velocity=6.7799634 -> lower=-0.523599 upper=0.785398 effort=25.76 velocity=2.1
- joint LAnkleRoll: limit lower=-0.349065844444444 upper=0.349065844444444 effort=27.911346822 velocity=10.28929 -> lower=-0.349066 upper=0.349066 effort=25.76 velocity=2.1
- joint LElbowRoll: limit lower=-2.60054054111111 upper=1.39626337777778 effort=13.820682 velocity=10.333784 -> lower=-2.0944 upper=2.0944 effort=7.404 velocity=3.7; origin xyz=0.205 0 0 rpy=0 0 0 -> xyz=0.205 0 0 rpy=0.17452 -0 0
- joint LElbowYaw: limit lower=-1.5707963 upper=0.401425721111111 effort=13.757736 velocity=10.3810644 -> lower=-1.5708 upper=0 effort=6.02 velocity=4
- joint LEyePitch: limit lower=-0.349065844444444 upper=0.349065844444444 effort=0 velocity=0 -> lower=-0.349066 upper=0.349066 effort=0.01752 velocity=293.215; parent LEyePitch_link -> LEyeYawLink
- joint LEyeYaw: child LEyePitch_link -> LEyeYawLink; limit lower=-0.523598766666667 upper=0.523598766666667 effort=0 velocity=0 -> lower=-0.523599 upper=0.523599 effort=0.01752 velocity=293.215; origin xyz=0 0.0325 0 rpy=0 0 0 -> xyz=0 0.03192 0 rpy=0 0 0
- joint LHipPitch: limit lower=-1.71042263777778 upper=0.523598766666667 effort=42.35835006 velocity=6.7799634 -> lower=-1.71042 upper=0.401426 effort=46.6 velocity=2.09
- joint LHipRoll: limit lower=-0.261799383333333 upper=0.523598766666667 effort=27.911346822 velocity=10.289294 -> lower=-0.261799 upper=0.523599 effort=46.6 velocity=2.09
- joint LHipYaw: limit lower=-0.261799383333333 upper=0.261799383333333 effort=17.754 velocity=8.082461 -> lower=-0.261799 upper=0.261799 effort=9.2 velocity=0.32
- joint LKneePitch: limit lower=-0.0523598766666667 upper=2.25147469666667 effort=17.350636374 velocity=8.27600953 -> lower=0 upper=2.00713 effort=38.17 velocity=6
- joint LShoulderPitch: limit lower=-1.51843642333333 upper=2.09439506666667 effort=21.882612 velocity=6.52664058 -> lower=-1.44478 upper=2.22041 effort=19.095 velocity=2.2; origin xyz=0.005 0.19 0 rpy=0 0 0 -> xyz=0.005 0.19 0 rpy=-0.158879 -0.0725189 -0.424682
- joint LShoulderYaw: limit lower=-0.200712860555556 upper=1.43989660833333 effort=13.820682 velocity=10.333784 -> lower=-0.430472 upper=1.14032 effort=9.031 velocity=4; origin xyz=0 0 0 rpy=0 0 0 -> xyz=0 0 0 rpy=0 0 0.430457
- joint LWristPitch: axis 0 0 1 -> 0 1 0; limit lower=-0.977384364444444 upper=0.977384364444444 effort=0 velocity=0 -> lower=-0.977384 upper=0.977384 effort=0.6 velocity=3.75
- joint LWristRoll: limit lower=-3.66519136666667 upper=0.523598766666667 effort=0 velocity=0 -> lower=-3.66519 upper=0.523599 effort=2.177 velocity=1.1; origin xyz=0.182 0 0 rpy=0 0 0 -> xyz=0.1823 0 0 rpy=0 0 0
- joint LWristYaw: axis 0 1 0 -> 0 0 1; limit lower=-0.488692182222222 upper=0.488692182222222 effort=0 velocity=0 -> lower=-0.436332 upper=0.436332 effort=0.862 velocity=2.26
- joint NeckPitch: limit lower=-0.698131688888889 upper=0.698131688888889 effort=23.115708 velocity=6.17848 -> lower=-0.349066 upper=0.698132 effort=2.978 velocity=2.2
- joint NeckYaw: limit lower=-1.5707963 upper=1.5707963 effort=24.2532552 velocity=5.8886917 -> lower=-1.5708 upper=1.5708 effort=3.662 velocity=4
- joint RAnklePitch: limit lower=-0.78539815 upper=0.523598766666667 effort=42.35835006 velocity=6.7799634 -> lower=-0.523599 upper=0.785398 effort=25.76 velocity=2.1
- joint RAnkleRoll: limit lower=-0.349065844444444 upper=0.349065844444444 effort=27.911346822 velocity=10.28929 -> lower=-0.349066 upper=0.349066 effort=25.76 velocity=2.1
- joint RElbowRoll: limit lower=-1.39626337777778 upper=2.60054054111111 effort=13.820682 velocity=10.333784 -> lower=-2.0944 upper=2.0944 effort=7.404 velocity=3.7; origin xyz=0.205 0 0 rpy=0 0 0 -> xyz=0.205 0 0 rpy=-0.17452 -0 0
- joint RElbowYaw: limit lower=-0.401425721111111 upper=1.5707963 effort=13.757736 velocity=10.3810644 -> lower=0 upper=1.5708 effort=6.02 velocity=4
- joint REyePitch: limit lower=-0.349065844444444 upper=0.349065844444444 effort=0 velocity=0 -> lower=-0.349066 upper=0.349066 effort=0.01752 velocity=293.215; parent REyePitch_link -> REyeYawLink
- joint REyeYaw: child REyePitch_link -> REyeYawLink; limit lower=-0.523598766666667 upper=0.523598766666667 effort=0 velocity=0 -> lower=-0.523599 upper=0.523599 effort=0.01752 velocity=293.215; origin xyz=0 -0.0325 0 rpy=0 0 0 -> xyz=0 -0.03192 0 rpy=0 0 0
- joint RHipPitch: limit lower=-1.71042263777778 upper=0.523598766666667 effort=42.35835006 velocity=6.7799634 -> lower=-1.71042 upper=0.401426 effort=46.6 velocity=2.09
- joint RHipRoll: limit lower=-0.523598766666667 upper=0.261799383333333 effort=27.911346822 velocity=10.289294 -> lower=-0.523599 upper=0.261799 effort=46.6 velocity=2.09
- joint RHipYaw: limit lower=-0.261799383333333 upper=0.261799383333333 effort=17.754 velocity=8.082461 -> lower=-0.261799 upper=0.261799 effort=9.2 velocity=0.32
- joint RKneePitch: limit lower=-0.0523598766666667 upper=2.25147469666667 effort=17.350636374 velocity=8.27600953 -> lower=0 upper=2.00713 effort=38.17 velocity=6
- joint RShoulderPitch: limit lower=-1.51843642333333 upper=2.09439506666667 effort=21.882612 velocity=6.52664058 -> lower=-1.44478 upper=2.22041 effort=19.095 velocity=2.2; origin xyz=0.005 -0.19 0 rpy=0 0 0 -> xyz=0.005 -0.19 0 rpy=0.158879 -0.0725189 0.424682
- joint RShoulderYaw: limit lower=-1.43989660833333 upper=0.200712860555556 effort=13.820682 velocity=10.333784 -> lower=-1.14032 upper=0.430472 effort=9.031 velocity=4; origin xyz=0 0 0 rpy=0 0 0 -> xyz=0 0 0 rpy=-0 -0 -0.430457
- joint RWristPitch: axis 0 0 1 -> 0 1 0; limit lower=-0.977384364444444 upper=0.977384364444444 effort=0 velocity=0 -> lower=-0.977384 upper=0.977384 effort=0.6 velocity=3.75
- joint RWristRoll: limit lower=-0.523598766666667 upper=3.66519136666667 effort=0 velocity=0 -> lower=-0.523599 upper=3.66519 effort=2.177 velocity=1.1; origin xyz=0.182 0 0 rpy=0 0 0 -> xyz=0.1823 0 0 rpy=0 0 0
- joint RWristYaw: axis 0 1 0 -> 0 0 1; limit lower=-0.488692182222222 upper=0.488692182222222 effort=0 velocity=0 -> lower=-0.436332 upper=0.436332 effort=0.862 velocity=2.26
- joint TrunkYaw: limit lower=-0.78539815 upper=0.78539815 effort=0 velocity=0 -> lower=-0.785398 upper=0.785398 effort=80.902 velocity=1.5; origin xyz=-0 -0 0.2 rpy=0 0 0 -> xyz=0 0 0.2 rpy=0 0 0
- joint gaze_joint: origin xyz=0.1111 0 0.0515 rpy=0 0 0 -> xyz=0.09178 0 0.05425 rpy=0 0 0

File: romeo_description/urdf/romeo_small.urdf (robot description, URDF)
Before this commit: robot romeo, 46 links, 45 joints
Links:
- removed link LEyePitch_link
- removed link REyePitch_link
- added link LEyeYawLink
- added link REyeYawLink
- link RElbowYawLink: mass 0.31403 -> 0.31265
- link RShoulderYawLink: mass 0.57071 -> 0.57151
- link l_ankle: mass 0.64224 -> 0.74347
- link l_toe: mass 0.2889 -> 0.24032
- link r_ankle: mass 0.64224 -> 0.74347
- link r_toe: mass 0.2889 -> 0.24032
Joints:
- joint HeadPitch: limit lower=-0.289724650888889 upper=0.349065844444444 effort=14.6811456 velocity=7.2988824 -> lower=-0.349066 upper=0.279253 effort=2.57 velocity=1.9
- joint HeadRoll: limit lower=-0.523598766666667 upper=0.523598766666667 effort=22.586421 velocity=4.7442645 -> lower=-0.349066 upper=0.349066 effort=0.9 velocity=1.5
- joint LAnklePitch: limit lower=-0.78539815 upper=0.523598766666667 effort=42.35835006 velocity=6.7799634 -> lower=-0.523599 upper=0.785398 effort=25.76 velocity=2.1
- joint LAnkleRoll: limit lower=-0.349065844444444 upper=0.349065844444444 effort=27.911346822 velocity=10.28929 -> lower=-0.349066 upper=0.349066 effort=25.76 velocity=2.1
- joint LElbowRoll: limit lower=-2.60054054111111 upper=1.39626337777778 effort=13.820682 velocity=10.333784 -> lower=-2.0944 upper=2.0944 effort=7.404 velocity=3.7; origin xyz=0.205 0 0 rpy=0 0 0 -> xyz=0.205 0 0 rpy=0.17452 -0 0
- joint LElbowYaw: limit lower=-1.5707963 upper=0.401425721111111 effort=13.757736 velocity=10.3810644 -> lower=-1.5708 upper=0 effort=6.02 velocity=4
- joint LEyePitch: limit lower=-0.349065844444444 upper=0.349065844444444 effort=0 velocity=0 -> lower=-0.349066 upper=0.349066 effort=0.01752 velocity=293.215; parent LEyePitch_link -> LEyeYawLink
- joint LEyeYaw: child LEyePitch_link -> LEyeYawLink; limit lower=-0.523598766666667 upper=0.523598766666667 effort=0 velocity=0 -> lower=-0.523599 upper=0.523599 effort=0.01752 velocity=293.215; origin xyz=0 0.0325 0 rpy=0 0 0 -> xyz=0 0.03192 0 rpy=0 0 0
- joint LHipPitch: limit lower=-1.71042263777778 upper=0.523598766666667 effort=42.35835006 velocity=6.7799634 -> lower=-1.71042 upper=0.401426 effort=46.6 velocity=2.09
- joint LHipRoll: limit lower=-0.261799383333333 upper=0.523598766666667 effort=27.911346822 velocity=10.289294 -> lower=-0.261799 upper=0.523599 effort=46.6 velocity=2.09
- joint LHipYaw: limit lower=-0.261799383333333 upper=0.261799383333333 effort=17.754 velocity=8.082461 -> lower=-0.261799 upper=0.261799 effort=9.2 velocity=0.32
- joint LKneePitch: limit lower=-0.0523598766666667 upper=2.25147469666667 effort=17.350636374 velocity=8.27600953 -> lower=0 upper=2.00713 effort=38.17 velocity=6
- joint LShoulderPitch: limit lower=-1.51843642333333 upper=2.09439506666667 effort=21.882612 velocity=6.52664058 -> lower=-1.44478 upper=2.22041 effort=19.095 velocity=2.2; origin xyz=0.005 0.19 0 rpy=0 0 0 -> xyz=0.005 0.19 0 rpy=-0.158879 -0.0725189 -0.424682
- joint LShoulderYaw: limit lower=-0.200712860555556 upper=1.43989660833333 effort=13.820682 velocity=10.333784 -> lower=-0.430472 upper=1.14032 effort=9.031 velocity=4; origin xyz=0 0 0 rpy=0 0 0 -> xyz=0 0 0 rpy=0 0 0.430457
- joint LWristPitch: axis 0 0 1 -> 0 1 0; limit lower=-0.977384364444444 upper=0.977384364444444 effort=0 velocity=0 -> lower=-0.977384 upper=0.977384 effort=0.6 velocity=3.75
- joint LWristRoll: limit lower=-3.66519136666667 upper=0.523598766666667 effort=0 velocity=0 -> lower=-3.66519 upper=0.523599 effort=2.177 velocity=1.1; origin xyz=0.182 0 0 rpy=0 0 0 -> xyz=0.1823 0 0 rpy=0 0 0
- joint LWristYaw: axis 0 1 0 -> 0 0 1; limit lower=-0.488692182222222 upper=0.488692182222222 effort=0 velocity=0 -> lower=-0.436332 upper=0.436332 effort=0.862 velocity=2.26
- joint NeckPitch: limit lower=-0.698131688888889 upper=0.698131688888889 effort=23.115708 velocity=6.17848 -> lower=-0.349066 upper=0.698132 effort=2.978 velocity=2.2
- joint NeckYaw: limit lower=-1.5707963 upper=1.5707963 effort=24.2532552 velocity=5.8886917 -> lower=-1.5708 upper=1.5708 effort=3.662 velocity=4
- joint RAnklePitch: limit lower=-0.78539815 upper=0.523598766666667 effort=42.35835006 velocity=6.7799634 -> lower=-0.523599 upper=0.785398 effort=25.76 velocity=2.1
- joint RAnkleRoll: limit lower=-0.349065844444444 upper=0.349065844444444 effort=27.911346822 velocity=10.28929 -> lower=-0.349066 upper=0.349066 effort=25.76 velocity=2.1
- joint RElbowRoll: limit lower=-1.39626337777778 upper=2.60054054111111 effort=13.820682 velocity=10.333784 -> lower=-2.0944 upper=2.0944 effort=7.404 velocity=3.7; origin xyz=0.205 0 0 rpy=0 0 0 -> xyz=0.205 0 0 rpy=-0.17452 -0 0
- joint RElbowYaw: limit lower=-0.401425721111111 upper=1.5707963 effort=13.757736 velocity=10.3810644 -> lower=0 upper=1.5708 effort=6.02 velocity=4
- joint REyePitch: limit lower=-0.349065844444444 upper=0.349065844444444 effort=0 velocity=0 -> lower=-0.349066 upper=0.349066 effort=0.01752 velocity=293.215; parent REyePitch_link -> REyeYawLink
- joint REyeYaw: child REyePitch_link -> REyeYawLink; limit lower=-0.523598766666667 upper=0.523598766666667 effort=0 velocity=0 -> lower=-0.523599 upper=0.523599 effort=0.01752 velocity=293.215; origin xyz=0 -0.0325 0 rpy=0 0 0 -> xyz=0 -0.03192 0 rpy=0 0 0
- joint RHipPitch: limit lower=-1.71042263777778 upper=0.523598766666667 effort=42.35835006 velocity=6.7799634 -> lower=-1.71042 upper=0.401426 effort=46.6 velocity=2.09
- joint RHipRoll: limit lower=-0.523598766666667 upper=0.261799383333333 effort=27.911346822 velocity=10.289294 -> lower=-0.523599 upper=0.261799 effort=46.6 velocity=2.09
- joint RHipYaw: limit lower=-0.261799383333333 upper=0.261799383333333 effort=17.754 velocity=8.082461 -> lower=-0.261799 upper=0.261799 effort=9.2 velocity=0.32
- joint RKneePitch: limit lower=-0.0523598766666667 upper=2.25147469666667 effort=17.350636374 velocity=8.27600953 -> lower=0 upper=2.00713 effort=38.17 velocity=6
- joint RShoulderPitch: limit lower=-1.51843642333333 upper=2.09439506666667 effort=21.882612 velocity=6.52664058 -> lower=-1.44478 upper=2.22041 effort=19.095 velocity=2.2; origin xyz=0.005 -0.19 0 rpy=0 0 0 -> xyz=0.005 -0.19 0 rpy=0.158879 -0.0725189 0.424682
- joint RShoulderYaw: limit lower=-1.43989660833333 upper=0.200712860555556 effort=13.820682 velocity=10.333784 -> lower=-1.14032 upper=0.430472 effort=9.031 velocity=4; origin xyz=0 0 0 rpy=0 0 0 -> xyz=0 0 0 rpy=-0 -0 -0.430457
- joint RWristPitch: axis 0 0 1 -> 0 1 0; limit lower=-0.977384364444444 upper=0.977384364444444 effort=0 velocity=0 -> lower=-0.977384 upper=0.977384 effort=0.6 velocity=3.75
- joint RWristRoll: limit lower=-0.523598766666667 upper=3.66519136666667 effort=0 velocity=0 -> lower=-0.523599 upper=3.66519 effort=2.177 velocity=1.1; origin xyz=0.182 0 0 rpy=0 0 0 -> xyz=0.1823 0 0 rpy=0 0 0
- joint RWristYaw: axis 0 1 0 -> 0 0 1; limit lower=-0.488692182222222 upper=0.488692182222222 effort=0 velocity=0 -> lower=-0.436332 upper=0.436332 effort=0.862 velocity=2.26
- joint TrunkYaw: limit lower=-0.78539815 upper=0.78539815 effort=0 velocity=0 -> lower=-0.785398 upper=0.785398 effort=80.902 velocity=1.5; origin xyz=-0 -0 0.2 rpy=0 0 0 -> xyz=0 0 0.2 rpy=0 0 0
- joint gaze_joint: origin xyz=0.1111 0 0.0515 rpy=0 0 0 -> xyz=0.09178 0 0.05425 rpy=0 0 0
