Commit message: Update romeo.urdf and romeo_small.urdf with 0.0.9 Aldebaran version

File: romeo_description/urdf/romeo.urdf (robot description, URDF)
Before this commit: robot romeo, 70 links, 69 joints
Links:
- removed link CameraLeft
- removed link CameraLeftEye
- removed link CameraRight
- removed link CameraRightEye
- removed link LEyePitch_link
- removed link REyePitch_link
- removed link l_toe
- removed link r_toe
- added link CameraDepth_frame
- added link CameraLeftEye_frame
- added link CameraLeft_frame
- added link CameraRightEye_frame
- added link CameraRight_frame
- added link HeadTouchFront_frame
- added link HeadTouchMiddle_frame
- added link HeadTouchRear_frame
- added link ImuHeadAccelerometer_frame
- added link ImuHeadGyrometer_frame
- added link ImuTorsoAccelerometer_frame
- added link ImuTorsoGyrometer_frame
- added link LFsrCenter_frame
- added link LFsrFL_frame
- added link LFsrFR_frame
- added link LFsrRCenter_frame
- added link RFsrCenter_frame
- added link RFsrFL_frame
- added link RFsrFR_frame
- added link RFsrRCenter_frame
- link HeadRollLink: geometry collision mesh filename=package://romeo_description/meshes/V1/collision/HeadRoll.dae scale=1 1 1; visual mesh filename=package://romeo_description/meshes/V1/visual/HeadRoll.dae scale=1 1 1
- link LElbowYawLink: geometry collision mesh filename=package://romeo_description/meshes/V1/collision/LElbowYaw.d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 scale=1 1 1; visual mesh filename=package://romeo_description/meshes/V1/visual/LElbowYaw.dae scale=1 1 1
- link LFinger11Link: geometry collision mesh filename=package://romeo_description/meshes/V1/collision/Phalax.dae; visual mesh filename=package://romeo_description/meshes/V1/visual/Phalax.dae
- link LFinger12Link: geometry collision mesh filename=package://romeo_description/meshes/V1/collision/Phalax.dae; visual mesh filename=package://romeo_description/meshes/V1/visual/Phalax.dae
- link LFinger13Link: geometry collision mesh filename=package://romeo_description/meshes/V1/collision/PhalaxEnd.d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; visual mesh filename=package://romeo_description/meshes/V1/visual/PhalaxEnd.dae
- link LFinger21Link: geometry collision mesh filename=package://romeo_description/meshes/V1/collision/Phalax.dae; visual mesh filename=package://romeo_description/meshes/V1/visual/Phalax.dae
- link LFinger22Link: geometry collision mesh filename=package://romeo_description/meshes/V1/collision/Phalax.dae; visual mesh filename=package://romeo_description/meshes/V1/visual/Phalax.dae
- link LFinger23Link: geometry collision mesh filename=package://romeo_description/meshes/V1/collision/PhalaxEnd.d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; visual mesh filename=package://romeo_description/meshes/V1/visual/PhalaxEnd.dae
- link LFinger31Link: geometry collision mesh filename=package://romeo_description/meshes/V1/collision/Phalax.dae; visual mesh filename=package://romeo_description/meshes/V1/visual/Phalax.dae
- link LFinger32Link: geometry collision mesh filename=package://romeo_description/meshes/V1/collision/Phalax.dae; visual mesh filename=package://romeo_description/meshes/V1/visual/Phalax.dae
- link LFinger33Link: geometry collision mesh filename=package://romeo_description/meshes/V1/collision/PhalaxEnd.d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; visual mesh filename=package://romeo_description/meshes/V1/visual/PhalaxEnd.dae
- link LHipPitchLink: geometry collision mesh filename=package://romeo_description/meshes/V1/collision/LHipPitch.d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 scale=1 1 1; visual mesh filename=package://romeo_description/meshes/V1/visual/LHipPitch.dae scale=1 1 1
- link LKneePitchLink: geometry collision mesh filename=package://romeo_description/meshes/V1/collision/LKneePitch.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 scale=1 1 1; visual mesh filename=package://romeo_description/meshes/V1/visual/LKneePitch.dae scale=1 1 1
- link LShoulderYawLink: geometry collision mesh filename=package://romeo_description/meshes/V1/collision/LShoulderYa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 scale=1 1 1; visual mesh filename=package://romeo_description/meshes/V1/visual/LShoulderYaw.d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 scale=1 1 1
- link LThumb1Link: geometry collision mesh filename=package://romeo_description/meshes/V1/collision/LThumb.dae; visual mesh filename=package://romeo_description/meshes/V1/visual/LThumb.dae
- link LThumb2Link: geometry collision mesh filename=package://romeo_description/meshes/V1/collision/Phalax.dae; visual mesh filename=package://romeo_description/meshes/V1/visual/Phalax.dae
- link LThumb3Link: geometry collision mesh filename=package://romeo_description/meshes/V1/collision/PhalaxEnd.d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; visual mesh filename=package://romeo_description/meshes/V1/visual/PhalaxEnd.dae
- link LWristRollLink: geometry collision mesh filename=package://romeo_description/meshes/V1/collision/LWristRoll.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 scale=1 1 1; visual mesh filename=package://romeo_description/meshes/V1/visual/LWristRoll.dae scale=1 1 1
- link LWristYawLink: geometry collision mesh filename=package://romeo_description/meshes/V1/collision/LWristYaw.d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 scale=1 1 1; visual mesh filename=package://romeo_description/meshes/V1/visual/LWristYaw.dae scale=1 1 1
- link NeckPitchLink: geometry collision mesh filename=package://romeo_description/meshes/V1/collision/NeckPitch.d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 scale=1 1 1; visual mesh filename=package://romeo_description/meshes/V1/visual/NeckPitch.dae scale=1 1 1
- link RElbowYawLink: mass 0.31403 -> 0.31265; geometry collision mesh filename=package://romeo_description/meshes/V1/collision/RElbowYaw.d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 scale=1 1 1; visual mesh filename=package://romeo_description/meshes/V1/visual/RElbowYaw.dae scale=1 1 1
- link RFinger11Link: geometry collision mesh filename=package://romeo_description/meshes/V1/collision/Phalax.dae; visual mesh filename=package://romeo_description/meshes/V1/visual/Phalax.dae
- link RFinger12Link: geometry collision mesh filename=package://romeo_description/meshes/V1/collision/Phalax.dae; visual mesh filename=package://romeo_description/meshes/V1/visual/Phalax.dae
- link RFinger13Link: geometry collision mesh filename=package://romeo_description/meshes/V1/collision/PhalaxEnd.d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; visual mesh filename=package://romeo_description/meshes/V1/visual/PhalaxEnd.dae
- link RFinger21Link: geometry collision mesh filename=package://romeo_description/meshes/V1/collision/Phalax.dae; visual mesh filename=package://romeo_description/meshes/V1/visual/Phalax.dae
- link RFinger22Link: geometry collision mesh filename=package://romeo_description/meshes/V1/collision/Phalax.dae; visual mesh filename=package://romeo_description/meshes/V1/visual/Phalax.dae
- link RFinger23Link: geometry collision mesh filename=package://romeo_description/meshes/V1/collision/PhalaxEnd.d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; visual mesh filename=package://romeo_description/meshes/V1/visual/PhalaxEnd.dae
- link RFinger31Link: geometry collision mesh filename=package://romeo_description/meshes/V1/collision/Phalax.dae; visual mesh filename=package://romeo_description/meshes/V1/visual/Phalax.dae
- link RFinger32Link: geometry collision mesh filename=package://romeo_description/meshes/V1/collision/Phalax.dae; visual mesh filename=package://romeo_description/meshes/V1/visual/Phalax.dae
- link RFinger33Link: geometry collision mesh filename=package://romeo_description/meshes/V1/collision/PhalaxEnd.d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; visual mesh filename=package://romeo_description/meshes/V1/visual/PhalaxEnd.dae
- link RHipPitchLink: geometry collision mesh filename=package://romeo_description/meshes/V1/collision/RHipPitch.d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 scale=1 1 1; visual mesh filename=package://romeo_description/meshes/V1/visual/RHipPitch.dae scale=1 1 1
- link RKneePitchLink: geometry collision mesh filename=package://romeo_description/meshes/V1/collision/RKneePitch.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 scale=1 1 1; visual mesh filename=package://romeo_description/meshes/V1/visual/RKneePitch.dae scale=1 1 1
- link RShoulderYawLink: mass 0.57071 -> 0.57151; geometry collision mesh filename=package://romeo_description/meshes/V1/collision/RShoulderYa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 scale=1 1 1; visual mesh filename=package://romeo_description/meshes/V1/visual/RShoulderYaw.d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 scale=1 1 1
- link RThumb1Link: geometry collision mesh filename=package://romeo_description/meshes/V1/collision/RThumb.dae; visual mesh filename=package://romeo_description/meshes/V1/visual/RThumb.dae
- link RThumb2Link: geometry collision mesh filename=package://romeo_description/meshes/V1/collision/Phalax.dae; visual mesh filename=package://romeo_description/meshes/V1/visual/Phalax.dae
- link RThumb3Link: geometry collision mesh filename=package://romeo_description/meshes/V1/collision/PhalaxEnd.d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; visual mesh filename=package://romeo_description/meshes/V1/visual/PhalaxEnd.dae
- link RWristRollLink: geometry collision mesh filename=package://romeo_description/meshes/V1/collision/RWristRoll.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 scale=1 1 1; visual mesh filename=package://romeo_description/meshes/V1/visual/RWristRoll.dae scale=1 1 1
- link RWristYawLink: geometry collision mesh filename=package://romeo_description/meshes/V1/collision/RWristYaw.d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 scale=1 1 1; visual mesh filename=package://romeo_description/meshes/V1/visual/RWristYaw.dae scale=1 1 1
- link body: geometry collision mesh filename=package://romeo_description/meshes/V1/collision/TrunkYaw.dae scale=1 1 1; visual mesh filename=package://romeo_description/meshes/V1/visual/TrunkYaw.dae scale=1 1 1
- link l_ankle: mass 0.64224 -> 1.07155; geometry collision mesh filename=package://romeo_description/meshes/V1/collision/LAnkleRoll.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 scale=1 1 1; visual mesh filename=package://romeo_description/meshes/V1/visual/LAnkleRoll.dae scale=1 1 1
- link l_wrist: geometry collision mesh filename=package://romeo_description/meshes/V1/collision/LWristPitch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 scale=1 1 1; visual mesh filename=package://romeo_description/meshes/V1/visual/LWristPitch.dae scale=1 1 1
- link r_ankle: mass 0.64224 -> 1.07155; geometry collision mesh filename=package://romeo_description/meshes/V1/collision/RAnkleRoll.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 scale=1 1 1; visual mesh filename=package://romeo_description/meshes/V1/visual/RAnkleRoll.dae scale=1 1 1
- link r_wrist: geometry collision mesh filename=package://romeo_description/meshes/V1/collision/RWristPitch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 scale=1 1 1; visual mesh filename=package://romeo_description/meshes/V1/visual/RWristPitch.dae scale=1 1 1
- link torso: geometry collision mesh filename=package://romeo_description/meshes/V1/collision/Torso.dae scale=1 1 1; visual mesh filename=package://romeo_description/meshes/V1/visual/Torso.dae scale=1 1 1
Joints:
- removed joint LEyePitch
- removed joint LEyeYaw
- removed joint LFinger11
- removed joint LToePitch
- removed joint REyePitch
- removed joint REyeYaw
- removed joint RFinger11
- removed joint RToePitch
- added joint CameraDepth_joint: type fixed, parent HeadRollLink, child CameraDepth_frame, origin xyz=0.1403 -0.04708 0.14655 rpy=2.0043951 0 1.57079632679
- added joint CameraLeftEye_joint: type fixed, parent HeadRollLink, child CameraLeftEye_frame, origin xyz=0.11017 0.03192 0.05426 rpy=0 0 0
- added joint CameraRightEye_joint: type fixed, parent HeadRollLink, child CameraRightEye_frame, origin xyz=0.11017 -0.03192 0.05426 rpy=0 0 0
- added joint HeadTouchFront_joint: type fixed, parent HeadRollLink, child HeadTouchFront_frame, origin xyz=0.0312 0 0.1014 rpy=0 -1.186099535 0
- added joint HeadTouchMiddle_joint: type fixed, parent HeadRollLink, child HeadTouchMiddle_frame, origin xyz=0.001 0 0.1099 rpy=0 -1.57079632679 0
- added joint HeadTouchRear_joint: type fixed, parent HeadRollLink, child HeadTouchRear_frame, origin xyz=-0.0257 0 0.1045 rpy=3.14159265359 -1.333192995 3.14159265359
- added joint ImuHeadAccelerometer_joint: type fixed, parent HeadRollLink, child ImuHeadAccelerometer_frame, origin xyz=-0.01135 -0.04225 0.16011 rpy=0 0 1.57079632679
- added joint ImuHeadGyrometer_joint: type fixed, parent HeadRollLink, child ImuHeadGyrometer_frame, origin xyz=-0.01135 -0.04225 0.16011 rpy=0 0 1.57079632679
- added joint ImuTorsoAccelerometer_joint: type fixed, parent body, child ImuTorsoAccelerometer_frame, origin xyz=0.06185 0.0087 -0.1582 rpy=0 0 0
- added joint ImuTorsoGyrometer_joint: type fixed, parent body, child ImuTorsoGyrometer_frame, origin xyz=0.06185 0.0087 -0.1582 rpy=0 0 0
- added joint LFsrCenter_joint: type fixed, parent l_ankle, child LFsrCenter_frame, origin xyz=0.073 0.02 -0.0646 rpy=0 0 0
- added joint LFsrFL_joint: type fixed, parent l_ankle, child LFsrFL_frame, origin xyz=0.13 0.0337 -0.0646 rpy=0 0 0
- added joint LFsrFR_joint: type fixed, parent l_ankle, child LFsrFR_frame, origin xyz=0.13 -0.0337 -0.0646 rpy=0 0 0
- added joint LFsrRCenter_joint: type fixed, parent l_ankle, child LFsrRCenter_frame, origin xyz=-0.04 0 -0.0646 rpy=0 0 0
- added joint LHand: type revolute, parent l_wrist, child LFinger11Link, origin xyz=0.10937 0.02468 0.00329 rpy=2.98023e-08 1.06465 0.122173, axis 0.121869 -0.992546 -4.37114e-08, limit lower=0.0 upper=1.0 effort=0 velocity=0
- added joint RFsrCenter_joint: type fixed, parent r_ankle, child RFsrCenter_frame, origin xyz=0.073 0.02 -0.0646 rpy=0 0 0
- added joint RFsrFL_joint: type fixed, parent r_ankle, child RFsrFL_frame, origin xyz=0.13 0.0337 -0.0646 rpy=0 0 0
- added joint RFsrFR_joint: type fixed, parent r_ankle, child RFsrFR_frame, origin xyz=0.13 -0.0337 -0.0646 rpy=0 0 0
- added joint RFsrRCenter_joint: type fixed, parent r_ankle, child RFsrRCenter_frame, origin xyz=-0.04 0 -0.0646 rpy=0 0 0
- added joint RHand: type revolute, parent r_wrist, child RFinger11Link, origin xyz=0.10937 -0.02468 0.00329 rpy=3.72529e-08 1.06465 -0.122173, axis -0.121869 -0.992546 -4.37114e-08, limit lower=-4.266806 upper=0.0 effort=0 velocity=0
- joint CameraLeft_joint: child CameraLeft -> CameraLeft_frame; origin xyz=-0.0021 0.055 0.0333 rpy=0 0 0 -> xyz=0.11999 0.04 0.09938 rpy=0 0 0; parent gaze -> HeadRollLink
- joint CameraRight_joint: child CameraRight -> CameraRight_frame; origin xyz=-0.0021 -0.055 0.0333 rpy=0 0 0 -> xyz=0.11999 -0.04 0.09938 rpy=0 0 0; parent gaze -> HeadRollLink
- joint HeadPitch: axis 0 1 0 -> 0 1.0 0; limit lower=-0.289724650888889 upper=0.349065844444444 effort=14.6811456 velocity=7.2988824 -> lower=-0.349066 upper=0.279253 effort=2.57 velocity=1.9
- joint HeadRoll: axis 1 0 0 -> 1.0 0 0; limit lower=-0.523598766666667 upper=0.523598766666667 effort=22.586421 velocity=4.7442645 -> lower=-0.349066 upper=0.349066 effort=0.9 velocity=1.5
- joint LAnklePitch: axis 0 1 0 -> 0 1.0 0; limit lower=-0.78539815 upper=0.523598766666667 effort=42.35835006 velocity=6.7799634 -> lower=-0.523599 upper=0.785398 effort=25.76 velocity=2.1
- joint LAnkleRoll: axis 1 0 0 -> 1.0 0 0; limit lower=-0.349065844444444 upper=0.349065844444444 effort=27.911346822 velocity=10.28929 -> lower=-0.349066 upper=0.349066 effort=25.76 velocity=2.1
- joint LElbowRoll: axis 1 0 0 -> 1.0 0 0; limit lower=-2.60054054111111 upper=1.39626337777778 effort=13.820682 velocity=10.333784 -> lower=-2.0944 upper=2.0944 effort=7.404 velocity=3.7; origin xyz=0.205 0 0 rpy=0 0 0 -> xyz=0.205 0 0 rpy=0.17452 0 0
- joint LElbowYaw: axis 0 0 1 -> 0 0 1.0; limit lower=-1.5707963 upper=0.401425721111111 effort=13.757736 velocity=10.3810644 -> lower=-1.5708 upper=0 effort=6.02 velocity=4.0
- joint LFinger12: mimic joint=LFinger11 multiplier=1 offset=0 -> joint=LHand multiplier=1 offset=0
- joint LFinger13: mimic joint=LFinger11 multiplier=1 offset=0 -> joint=LHand multiplier=1 offset=0
- joint LFinger21: mimic joint=LFinger11 multiplier=1 offset=0 -> joint=LHand multiplier=1 offset=0
- joint LFinger22: mimic joint=LFinger11 multiplier=1 offset=0 -> joint=LHand multiplier=1 offset=0
- joint LFinger23: mimic joint=LFinger11 multiplier=1 offset=0 -> joint=LHand multiplier=1 offset=0
- joint LFinger31: mimic joint=LFinger11 multiplier=1 offset=0 -> joint=LHand multiplier=1 offset=0
- joint LFinger32: mimic joint=LFinger11 multiplier=1 offset=0 -> joint=LHand multiplier=1 offset=0
- joint LFinger33: mimic joint=LFinger11 multiplier=1 offset=0 -> joint=LHand multiplier=1 offset=0
- joint LHipPitch: axis 0 1 0 -> 0 1.0 0; limit lower=-1.71042263777778 upper=0.523598766666667 effort=42.35835006 velocity=6.7799634 -> lower=-1.71042 upper=0.401426 effort=46.6 velocity=2.09
- joint LHipRoll: axis 1 0 0 -> 1.0 0 0; limit lower=-0.261799383333333 upper=0.523598766666667 effort=27.911346822 velocity=10.289294 -> lower=-0.261799 upper=0.523599 effort=46.6 velocity=2.09
- joint LHipYaw: axis 0 0 1 -> 0 0 1.0; limit lower=-0.261799383333333 upper=0.261799383333333 effort=17.754 velocity=8.082461 -> lower=-0.261799 upper=0.261799 effort=9.2 velocity=0.32
- joint LKneePitch: axis 0 1 0 -> 0 1.0 0; limit lower=-0.0523598766666667 upper=2.25147469666667 effort=17.350636374 velocity=8.27600953 -> lower=0 upper=2.00713 effort=38.17 velocity=6.0
- joint LShoulderPitch: axis 0 1 0 -> 0 1.0 0; limit lower=-1.51843642333333 upper=2.09439506666667 effort=21.882612 velocity=6.52664058 -> lower=-1.44478 upper=2.22041 effort=19.095 velocity=2.2; origin xyz=0.005 0.19 0 rpy=0 0 0 -> xyz=0.005 0.19 0 rpy=-0.158879 -0.0725189 -0.424682
- joint LShoulderYaw: axis 0 0 1 -> 0 0 1.0; limit lower=-0.200712860555556 upper=1.43989660833333 effort=13.820682 velocity=10.333784 -> lower=-0.430472 upper=1.14032 effort=9.031 velocity=4.0; origin xyz=0 0 0 rpy=0 0 0 -> xyz=0 0 0 rpy=0 0 0.430457
- joint LThumb1: mimic joint=LFinger11 multiplier=-1 offset=0 -> joint=LHand multiplier=-1 offset=0
- joint LThumb2: mimic joint=LFinger11 multiplier=1 offset=0 -> joint=LHand multiplier=1 offset=0
- joint LThumb3: mimic joint=LFinger11 multiplier=1 offset=0 -> joint=LHand multiplier=1 offset=0
- joint LWristPitch: axis 0 0 1 -> 0 1.0 0; limit lower=-0.977384364444444 upper=0.977384364444444 effort=0 velocity=0 -> lower=-0.977384 upper=0.977384 effort=0.6 velocity=3.75
- joint LWristRoll: axis 1 0 0 -> 1.0 0 0; limit lower=-3.66519136666667 upper=0.523598766666667 effort=0 velocity=0 -> lower=-3.66519 upper=0.523599 effort=2.177 velocity=1.1; origin xyz=0.182 0 0 rpy=0 0 0 -> xyz=0.1823 0 0 rpy=0 0 0
- joint LWristYaw: axis 0 1 0 -> 0 0 1.0; limit lower=-0.488692182222222 upper=0.488692182222222 effort=0 velocity=0 -> lower=-0.436332 upper=0.436332 effort=0.862 velocity=2.26
- joint NeckPitch: axis 0 1 0 -> 0 1.0 0; limit lower=-0.698131688888889 upper=0.698131688888889 effort=23.115708 velocity=6.17848 -> lower=-0.349066 upper=0.698132 effort=2.978 velocity=2.2
- joint NeckYaw: axis 0 0 1 -> 0 0 1.0; limit lower=-1.5707963 upper=1.5707963 effort=24.2532552 velocity=5.8886917 -> lower=-1.5708 upper=1.5708 effort=3.662 velocity=4.0
- joint RAnklePitch: axis 0 1 0 -> 0 1.0 0; limit lower=-0.78539815 upper=0.523598766666667 effort=42.35835006 velocity=6.7799634 -> lower=-0.523599 upper=0.785398 effort=25.76 velocity=2.1
- joint RAnkleRoll: axis 1 0 0 -> 1.0 0 0; limit lower=-0.349065844444444 upper=0.349065844444444 effort=27.911346822 velocity=10.28929 -> lower=-0.349066 upper=0.349066 effort=25.76 velocity=2.1
- joint RElbowRoll: axis 1 0 0 -> 1.0 0 0; limit lower=-1.39626337777778 upper=2.60054054111111 effort=13.820682 velocity=10.333784 -> lower=-2.0944 upper=2.0944 effort=7.404 velocity=3.7; origin xyz=0.205 0 0 rpy=0 0 0 -> xyz=0.205 0 0 rpy=-0.17452 0 0
- joint RElbowYaw: axis 0 0 1 -> 0 0 1.0; limit lower=-0.401425721111111 upper=1.5707963 effort=13.757736 velocity=10.3810644 -> lower=0 upper=1.5708 effort=6.02 velocity=4.0
- joint RFinger12: mimic joint=RFinger11 multiplier=1 offset=0 -> joint=RHand multiplier=1 offset=0
- joint RFinger13: mimic joint=RFinger11 multiplier=1 offset=0 -> joint=RHand multiplier=1 offset=0
- joint RFinger21: mimic joint=RFinger11 multiplier=1 offset=0 -> joint=RHand multiplier=1 offset=0
- joint RFinger22: mimic joint=RFinger11 multiplier=1 offset=0 -> joint=RHand multiplier=1 offset=0
- joint RFinger23: mimic joint=RFinger11 multiplier=1 offset=0 -> joint=RHand multiplier=1 offset=0
- joint RFinger31: mimic joint=RFinger11 multiplier=1 offset=0 -> joint=RHand multiplier=1 offset=0
- joint RFinger32: mimic joint=RFinger11 multiplier=1 offset=0 -> joint=RHand multiplier=1 offset=0
- joint RFinger33: mimic joint=RFinger11 multiplier=1 offset=0 -> joint=RHand multiplier=1 offset=0
- joint RHipPitch: axis 0 1 0 -> 0 1.0 0; limit lower=-1.71042263777778 upper=0.523598766666667 effort=42.35835006 velocity=6.7799634 -> lower=-1.71042 upper=0.401426 effort=46.6 velocity=2.09
- joint RHipRoll: axis 1 0 0 -> 1.0 0 0; limit lower=-0.523598766666667 upper=0.261799383333333 effort=27.911346822 velocity=10.289294 -> lower=-0.523599 upper=0.261799 effort=46.6 velocity=2.09
- joint RHipYaw: axis 0 0 1 -> 0 0 1.0; limit lower=-0.261799383333333 upper=0.261799383333333 effort=17.754 velocity=8.082461 -> lower=-0.261799 upper=0.261799 effort=9.2 velocity=0.32
- joint RKneePitch: axis 0 1 0 -> 0 1.0 0; limit lower=-0.0523598766666667 upper=2.25147469666667 effort=17.350636374 velocity=8.27600953 -> lower=0 upper=2.00713 effort=38.17 velocity=6.0
- joint RShoulderPitch: axis 0 1 0 -> 0 1.0 0; limit lower=-1.51843642333333 upper=2.09439506666667 effort=21.882612 velocity=6.52664058 -> lower=-1.44478 upper=2.22041 effort=19.095 velocity=2.2; origin xyz=0.005 -0.19 0 rpy=0 0 0 -> xyz=0.005 -0.19 0 rpy=0.158879 -0.0725189 0.424682
- joint RShoulderYaw: axis 0 0 1 -> 0 0 1.0; limit lower=-1.43989660833333 upper=0.200712860555556 effort=13.820682 velocity=10.333784 -> lower=-1.14032 upper=0.430472 effort=9.031 velocity=4.0; origin xyz=0 0 0 rpy=0 0 0 -> xyz=0 0 0 rpy=0 0 -0.430457
- joint RThumb1: mimic joint=RFinger11 multiplier=-1 offset=0 -> joint=RHand multiplier=-1 offset=0
- joint RThumb2: mimic joint=RFinger11 multiplier=1 offset=0 -> joint=RHand multiplier=1 offset=0
- joint RThumb3: mimic joint=RFinger11 multiplier=1 offset=0 -> joint=RHand multiplier=1 offset=0
- joint RWristPitch: axis 0 0 1 -> 0 1.0 0; limit lower=-0.977384364444444 upper=0.977384364444444 effort=0 velocity=0 -> lower=-0.977384 upper=0.977384 effort=0.6 velocity=3.75
- joint RWristRoll: axis 1 0 0 -> 1.0 0 0; limit lower=-0.523598766666667 upper=3.66519136666667 effort=0 velocity=0 -> lower=-0.523599 upper=3.66519 effort=2.177 velocity=1.1; origin xyz=0.182 0 0 rpy=0 0 0 -> xyz=0.1823 0 0 rpy=0 0 0
- joint RWristYaw: axis 0 1 0 -> 0 0 1.0; limit lower=-0.488692182222222 upper=0.488692182222222 effort=0 velocity=0 -> lower=-0.436332 upper=0.436332 effort=0.862 velocity=2.26
- joint TrunkYaw: axis 0 0 1 -> 0 0 1.0; limit lower=-0.78539815 upper=0.78539815 effort=0 velocity=0 -> lower=-0.785398 upper=0.785398 effort=80.902 velocity=1.5; origin xyz=-0 -0 0.2 rpy=0 0 0 -> xyz=0 0 0.2 rpy=0 0 0
- joint gaze_joint: origin xyz=0.1111 0 0.0515 rpy=0 0 0 -> xyz=0.11017 0 0.05426 rpy=0 0 0
- joint l_sole_joint: origin xyz=0 0 -0.067 rpy=0 0 0 -> xyz=0 0 -0.0684 rpy=0 0 0
- joint r_sole_joint: origin xyz=0 0 -0.067 rpy=0 0 0 -> xyz=0 0 -0.0684 rpy=0 0 0
